Commit message: adds tf_prefix argument to imu.gazebo.urdf.xacro

File: mir_description/urdf/include/imu.gazebo.urdf.xacro (robot description, xacro)
@@ -1,4 +1,12 @@
 <?xml version="1.0"?>
 <robot xmlns:xacro="http://ros.org/wiki/xacro">
+  <!-- If tf_prefix is given, use "frame tf_prefix/imu_frame", else "imu_frame" -->
+  <xacro:arg name="tf_prefix" default="" />
+  <xacro:if value="$(eval tf_prefix == '')">
+      <xacro:property name="imu_frame" value="imu_frame" />
+  </xacro:if>
+  <xacro:unless value="$(eval tf_prefix == '')">
+      <xacro:property name="imu_frame" value="$(arg tf_prefix)/imu_frame" />
+  </xacro:unless>
   <xacro:macro name="imu_gazebo" params="link imu_topic update_rate stdev">
     <gazebo reference="${link}">
@@ -16,5 +24,5 @@
           <xyzOffset>0 0 0</xyzOffset>
           <rpyOffset>0 0 0</rpyOffset>
-          <frameName>imu_frame</frameName>  <!-- from real MiR -->
+          <frameName>${imu_frame}</frameName>  <!-- from real MiR -->
         </plugin>
         <pose>0 0 0 0 0 0</pose>

Commit message: workaround eval in xacro for indigo support

File: mir_description/urdf/include/imu.gazebo.urdf.xacro (robot description, xacro)
@@ -3,8 +3,9 @@
   <!-- If tf_prefix is given, use "frame tf_prefix/imu_frame", else "imu_frame" -->
   <xacro:arg name="tf_prefix" default="" />
-  <xacro:if value="$(eval tf_prefix == '')">
+  <xacro:property name="tf_prefix" value="$(arg tf_prefix)" />
+  <xacro:if value="${tf_prefix == ''}">
       <xacro:property name="imu_frame" value="imu_frame" />
   </xacro:if>
-  <xacro:unless value="$(eval tf_prefix == '')">
+  <xacro:unless value="${tf_prefix == ''}">
       <xacro:property name="imu_frame" value="$(arg tf_prefix)/imu_frame" />
   </xacro:unless>

Commit message: added prefix/namespace possibility to mir_description

File: mir_description/urdf/include/imu.gazebo.urdf.xacro (robot description, xacro)
@@ -74,5 +74,5 @@
         <initial_orientation_as_reference>false</initial_orientation_as_reference>
           <ros>
-            <namespace>/${imu_topic}</namespace>
+            <namespace>${imu_topic}</namespace>
             <remapping>~/out:=data</remapping>
             <frame_name>${imu_frame}</frame_name>  <!-- from real MiR -->

File: mir_description/urdf/include/mir_100.gazebo.xacro (robot description, xacro)
@@ -2,8 +2,11 @@
 <robot xmlns:xacro="http://ros.org/wiki/xacro">
   <!-- See https://github.com/ros-simulation/gazebo_ros_pkgs/wiki/ROS-2-Migration:-Diff-drive for ros2 information -->
-  <xacro:macro name="diff_controller_plugin_gazebo" params="prefix left_wheel_joint right_wheel_joint wheel_separation wheel_radius">
+  <xacro:macro name="diff_controller_plugin_gazebo" params="prefix namespace left_wheel_joint right_wheel_joint wheel_separation wheel_radius">
     <gazebo>
       <!-- Use gazebo_ros_joint_state_publisher instead of publishWheelJointState -->
       <plugin name="joint_states" filename="libgazebo_ros_joint_state_publisher.so">
+        <ros>
+          <namespace>${namespace}</namespace>
+        </ros>
         <update_rate>1000.0</update_rate>
         <joint_name>${right_wheel_joint}</joint_name>
@@ -12,5 +15,5 @@
       <plugin name="diff_drive_controller" filename="libgazebo_ros_diff_drive.so">
         <ros>
-          <namespace>/mobile_base_controller</namespace>
+          <namespace>${prefix}mobile_base_controller</namespace>
         </ros>
         <legacy_mode>false</legacy_mode>
@@ -21,6 +24,6 @@
         <wheel_separation>${wheel_separation}</wheel_separation>
         <wheel_diameter>${2*wheel_radius}</wheel_diameter>
-        <odometry_frame>odom</odometry_frame>
-        <robot_base_frame>base_footprint</robot_base_frame>
+        <odometry_frame>${prefix}odom</odometry_frame>
+        <robot_base_frame>${prefix}base_footprint</robot_base_frame>
         <publish_odom>true</publish_odom>
         <publish_wheel_tf>false</publish_wheel_tf>
@@ -49,8 +52,9 @@
   </xacro:macro>
  <!-- See https://github.com/ros-simulation/gazebo_ros_pkgs/wiki/ROS-2-Migration:-P3D for ros2 information -->
-  <xacro:macro name="p3d_base_controller" params="prefix">
+  <xacro:macro name="p3d_base_controller" params="namespace prefix">
     <gazebo>
       <plugin name="p3d_base_controller" filename="libgazebo_ros_p3d.so">
         <ros>
+          <namespace>${namespace}</namespace>
           <remapping>odom:=base_pose_ground_truth</remapping>
         </ros>

File: mir_description/urdf/include/mir_100_v1.urdf.xacro (robot description, xacro)
@@ -24,5 +24,5 @@
   <xacro:property name="mir_100_caster_wheel_base_dz" value="${mir_100_caster_wheel_radius-mir_100_caster_wheel_dz}" />
   <xacro:property name="imu_stdev" value="0.00017" />
-  <xacro:macro name="actuated_wheel" params="prefix locationprefix locationright">
+  <xacro:macro name="actuated_wheel" params="prefix namespace locationprefix locationright">
     <joint name="${prefix}${locationprefix}_wheel_joint" type="continuous">
       <origin xyz="0.0 ${-mir_100_act_wheel_dy * locationright} ${mir_100_act_wheel_radius}" rpy="0 0 0" />
@@ -64,5 +64,7 @@
     </joint>
     <gazebo>
-      <plugin name="joint_states" filename="libgazebo_ros_joint_state_publisher.so">
+      <plugin name="${locationprefix}_caster_rotation_joint_states" filename="libgazebo_ros_joint_state_publisher.so">
+        <ros>
+        </ros>
         <update_rate>200.0</update_rate>
         <joint_name>${prefix}${locationprefix}_caster_rotation_joint</joint_name>
@@ -107,5 +109,8 @@
     </joint>
     <gazebo>
-      <plugin name="joint_states" filename="libgazebo_ros_joint_state_publisher.so">
+      <plugin name="${locationprefix}_caster_wheel_joint_states" filename="libgazebo_ros_joint_state_publisher.so">
+        <ros>
+          <namespace>${namespace}</namespace>
+        </ros>
         <update_rate>200.0</update_rate>
         <joint_name>${prefix}${locationprefix}_caster_wheel_joint</joint_name>
@@ -134,5 +139,5 @@
     </gazebo>
   </xacro:macro>
-  <xacro:macro name="mir_100" params="prefix">
+  <xacro:macro name="mir_100" params="prefix namespace">
     <link name="${prefix}base_footprint" />
     <joint name="${prefix}base_joint" type="fixed">
@@ -169,5 +174,5 @@
     </joint>
     <link name="${prefix}imu_link" />
-    <xacro:imu_gazebo link="${prefix}imu_link" imu_topic="imu_data" update_rate="50.0" stdev="${imu_stdev}" />
+    <xacro:imu_gazebo link="${prefix}imu_link" imu_topic="${prefix}imu_data" update_rate="50.0" stdev="${imu_stdev}" />
     <!-- Create an alias for imu_link. This is necessary because the real MiR's
          TF has imu_link, but the imu_data topic is published in the imu_frame
@@ -185,5 +190,5 @@
       <origin xyz="0.4288 0.2358 0.1914" rpy="0.0 0.0 ${0.25 * pi}" />  <!-- from visually matching up the meshes of the MiR and the laser scanner -->
     </joint>
-    <xacro:sick_s300 prefix="${prefix}" link="front_laser_link" topic="f_scan" />
+    <xacro:sick_s300 prefix="${prefix}" namespace="${namespace}" link="front_laser_link" topic="f_scan" />
     <joint name="${prefix}base_link_to_back_laser_joint" type="fixed">
       <parent link="${prefix}base_link" />
@@ -191,5 +196,5 @@
       <origin xyz="-0.3548 -0.2352 0.1914" rpy="0.0 0.0 ${-0.75 * pi}" />  <!-- from visually matching up the meshes of the MiR and the laser scanner -->
     </joint>
-    <xacro:sick_s300 prefix="${prefix}" link="back_laser_link" topic="b_scan" />
+    <xacro:sick_s300 prefix="${prefix}" namespace="${namespace}" link="back_laser_link" topic="b_scan" />
     <!-- Ultrasound sensors -->
     <joint name="${prefix}us_1_joint" type="fixed">   <!-- right ultrasound -->
@@ -206,6 +211,6 @@
     <link name="${prefix}us_2_frame" />
     <!-- wheels -->
-    <xacro:actuated_wheel prefix="${prefix}" locationprefix="left" locationright="-1"/>
-    <xacro:actuated_wheel prefix="${prefix}" locationprefix="right" locationright="1"/>
+    <xacro:actuated_wheel prefix="${prefix}" namespace="${namespace}" locationprefix="left" locationright="-1"/>
+    <xacro:actuated_wheel prefix="${prefix}" namespace="${namespace}" locationprefix="right" locationright="1"/>
     <xacro:caster_wheel prefix="${prefix}" locationprefix="fl" locationright="-1" wheel_base_dx="${mir_100_front_caster_wheel_base_dx}"/>
     <xacro:caster_wheel prefix="${prefix}" locationprefix="fr" locationright="1" wheel_base_dx="${mir_100_front_caster_wheel_base_dx}"/>
@@ -222,5 +227,5 @@
     <!-- set the gazebo friction parameters for the wheels -->
     <xacro:set_all_wheel_frictions prefix="${prefix}"/>
-    <xacro:p3d_base_controller prefix="${prefix}" />
+    <xacro:p3d_base_controller prefix="${prefix}" namespace="${namespace}"/>
   </xacro:macro>
 </robot>

File: mir_description/urdf/include/sick_s300.urdf.xacro (robot description, xacro)
@@ -6,5 +6,5 @@
   <xacro:property name="laser_z" value="0.185" />
   <xacro:property name="laser_mass" value="2.0" />
-  <xacro:macro name="sick_s300" params="link topic prefix">
+  <xacro:macro name="sick_s300" params="link topic prefix namespace">
     <link name="${prefix}${link}">
       <visual>
@@ -58,4 +58,5 @@
           <ros>
             <remapping>~/out:=${topic}</remapping>
+            <namespace>${namespace}</namespace>
           </ros>
           <output_type>sensor_msgs/LaserScan</output_type>

File: mir_description/urdf/mir.urdf.xacro (robot description, xacro)
@@ -5,19 +5,22 @@
   <xacro:include filename="$(find mir_description)/urdf/include/mir_100_v1.urdf.xacro" />
   <xacro:include filename="$(find mir_description)/urdf/include/common.gazebo.xacro" />
+  <xacro:arg name="namespace" default=""/>
   <xacro:arg name="tf_prefix" default="" />
-  <xacro:property name="tf_prefix_" value="$(arg tf_prefix)" />
-  <xacro:if value="${tf_prefix_ == ''}">
+  <xacro:property name="tf_prefix_val" value="$(arg tf_prefix)" />
+  <xacro:if value="${tf_prefix_val == ''}">
     <xacro:property name="prefix" value="" />
+    <xacro:property name="namespace" value=""/>
   </xacro:if>
-  <xacro:unless value="${tf_prefix_ == ''}">
-    <xacro:property name="prefix" value="${tf_prefix_}/" />
+  <xacro:unless value="${tf_prefix_val == ''}">
+    <xacro:property name="prefix" value="${tf_prefix_val}/" />
+    <xacro:property name="namespace" value="${tf_prefix_val}"/>
   </xacro:unless>
-  <xacro:mir_100 prefix="${prefix}"/>
+  <xacro:mir_100 prefix="${prefix}" namespace="${namespace}"/>
   <!--
   <xacro:controller_plugin_gazebo robot_namespace=""/>
   -->
-  <xacro:diff_controller_plugin_gazebo prefix=""
-    left_wheel_joint="left_wheel_joint"
-    right_wheel_joint="right_wheel_joint"
+  <xacro:diff_controller_plugin_gazebo prefix="${prefix}" namespace="${namespace}"
+    left_wheel_joint="${prefix}left_wheel_joint"
+    right_wheel_joint="${prefix}right_wheel_joint"
     wheel_separation="${2*mir_100_act_wheel_dy}"
     wheel_radius="${mir_100_act_wheel_radius}"/>

Commit message: Add namespace support (#17)
* add namespace for simulation and teleop

* add namespace to gazebo entity

* change to prefix only in urdfs

* enable ns for joint_state_publisher

* add namespace support to mir_navigation + ns instructions to readme

* switched namespaces to remappings in urdfs

* resolved gazeboplugin namespace errors

* fixes for namespace support driver

* added navigation config namespace examples

* minor fixes for namespace launch and adaptions in rviz configs

* fixed tf namespace bug in driver

* split up of driver launch files

* fixed params filename + added namespace args in nav launch

* enabled qos settings for ros2 topics in driver

* removed unused rviz parameter

File: mir_description/urdf/include/imu.gazebo.urdf.xacro (robot description, xacro)
@@ -80,5 +80,4 @@
         </plugin>
       </sensor>
-      -->
     </gazebo>
   </xacro:macro>

File: mir_description/urdf/include/mir_100.gazebo.xacro (robot description, xacro)
@@ -2,10 +2,10 @@
 <robot xmlns:xacro="http://ros.org/wiki/xacro">
   <!-- See https://github.com/ros-simulation/gazebo_ros_pkgs/wiki/ROS-2-Migration:-Diff-drive for ros2 information -->
-  <xacro:macro name="diff_controller_plugin_gazebo" params="prefix namespace left_wheel_joint right_wheel_joint wheel_separation wheel_radius">
+  <xacro:macro name="diff_controller_plugin_gazebo" params="prefix ns left_wheel_joint right_wheel_joint wheel_separation wheel_radius">
     <gazebo>
       <!-- Use gazebo_ros_joint_state_publisher instead of publishWheelJointState -->
       <plugin name="joint_states" filename="libgazebo_ros_joint_state_publisher.so">
         <ros>
-          <namespace>${namespace}</namespace>
+          <namespace>${ns}</namespace>
         </ros>
         <update_rate>1000.0</update_rate>
@@ -15,5 +15,6 @@
       <plugin name="diff_drive_controller" filename="libgazebo_ros_diff_drive.so">
         <ros>
-          <namespace>${prefix}</namespace>
+          <remapping>cmd_vel:=${prefix}cmd_vel</remapping>
+          <remapping>odom:=${prefix}odom</remapping>
         </ros>
         <legacy_mode>false</legacy_mode>
@@ -52,10 +53,9 @@
   </xacro:macro>
  <!-- See https://github.com/ros-simulation/gazebo_ros_pkgs/wiki/ROS-2-Migration:-P3D for ros2 information -->
-  <xacro:macro name="p3d_base_controller" params="namespace prefix">
+  <xacro:macro name="p3d_base_controller" params="prefix">
     <gazebo>
       <plugin name="p3d_base_controller" filename="libgazebo_ros_p3d.so">
         <ros>
-          <namespace>${namespace}</namespace>
-          <remapping>odom:=base_pose_ground_truth</remapping>
+          <remapping>odom:=${prefix}base_pose_ground_truth</remapping>
         </ros>
         <always_on>true</always_on>

File: mir_description/urdf/include/mir_100_v1.urdf.xacro (robot description, xacro)
@@ -24,5 +24,5 @@
   <xacro:property name="mir_100_caster_wheel_base_dz" value="${mir_100_caster_wheel_radius-mir_100_caster_wheel_dz}" />
   <xacro:property name="imu_stdev" value="0.00017" />
-  <xacro:macro name="actuated_wheel" params="prefix namespace locationprefix locationright">
+  <xacro:macro name="actuated_wheel" params="prefix  locationprefix locationright">
     <joint name="${prefix}${locationprefix}_wheel_joint" type="continuous">
       <origin xyz="0.0 ${-mir_100_act_wheel_dy * locationright} ${mir_100_act_wheel_radius}" rpy="0 0 0" />
@@ -54,5 +54,5 @@
     </gazebo>
   </xacro:macro>
-  <xacro:macro name="caster_wheel" params="prefix locationprefix locationright wheel_base_dx">
+  <xacro:macro name="caster_wheel" params="prefix ns locationprefix locationright wheel_base_dx">
     <!-- caster hub -->
     <joint name="${prefix}${locationprefix}_caster_rotation_joint" type="continuous">
@@ -66,4 +66,5 @@
       <plugin name="${locationprefix}_caster_rotation_joint_states" filename="libgazebo_ros_joint_state_publisher.so">
         <ros>
+          <namespace>${ns}</namespace>
         </ros>
         <update_rate>200.0</update_rate>
@@ -111,5 +112,5 @@
       <plugin name="${locationprefix}_caster_wheel_joint_states" filename="libgazebo_ros_joint_state_publisher.so">
         <ros>
-          <namespace>${namespace}</namespace>
+          <namespace>${ns}</namespace>
         </ros>
         <update_rate>200.0</update_rate>
@@ -139,5 +140,5 @@
     </gazebo>
   </xacro:macro>
-  <xacro:macro name="mir_100" params="prefix namespace">
+  <xacro:macro name="mir_100" params="prefix ns">
     <link name="${prefix}base_footprint" />
     <joint name="${prefix}base_joint" type="fixed">
@@ -198,5 +199,5 @@
       <origin xyz="0.4288 0.2358 0.1914" rpy="0.0 0.0 ${0.25 * pi}" />  <!-- from visually matching up the meshes of the MiR and the laser scanner -->
     </joint>
-    <xacro:sick_s300 prefix="${prefix}" namespace="${namespace}" link="front_laser_link" topic="f_scan" />
+    <xacro:sick_s300 prefix="${prefix}" link="front_laser_link" topic="f_scan" />
     <joint name="${prefix}base_link_to_back_laser_joint" type="fixed">
       <parent link="${prefix}base_link" />
@@ -204,5 +205,5 @@
       <origin xyz="-0.3548 -0.2352 0.1914" rpy="0.0 0.0 ${-0.75 * pi}" />  <!-- from visually matching up the meshes of the MiR and the laser scanner -->
     </joint>
-    <xacro:sick_s300 prefix="${prefix}" namespace="${namespace}" link="back_laser_link" topic="b_scan" />
+    <xacro:sick_s300 prefix="${prefix}" link="back_laser_link" topic="b_scan" />
     <!-- Ultrasound sensors -->
     <joint name="${prefix}us_1_joint" type="fixed">   <!-- right ultrasound -->
@@ -219,10 +220,10 @@
     <link name="${prefix}us_2_frame" />
     <!-- wheels -->
-    <xacro:actuated_wheel prefix="${prefix}" namespace="${namespace}" locationprefix="left" locationright="-1"/>
-    <xacro:actuated_wheel prefix="${prefix}" namespace="${namespace}" locationprefix="right" locationright="1"/>
-    <xacro:caster_wheel prefix="${prefix}" locationprefix="fl" locationright="-1" wheel_base_dx="${mir_100_front_caster_wheel_base_dx}"/>
-    <xacro:caster_wheel prefix="${prefix}" locationprefix="fr" locationright="1" wheel_base_dx="${mir_100_front_caster_wheel_base_dx}"/>
-    <xacro:caster_wheel prefix="${prefix}" locationprefix="bl" locationright="-1" wheel_base_dx="${mir_100_back_caster_wheel_base_dx}"/>
-    <xacro:caster_wheel prefix="${prefix}" locationprefix="br" locationright="1" wheel_base_dx="${mir_100_back_caster_wheel_base_dx}"/>
+    <xacro:actuated_wheel prefix="${prefix}" locationprefix="left" locationright="-1"/>
+    <xacro:actuated_wheel prefix="${prefix}" locationprefix="right" locationright="1"/>
+    <xacro:caster_wheel prefix="${prefix}" ns="${ns}" locationprefix="fl" locationright="-1" wheel_base_dx="${mir_100_front_caster_wheel_base_dx}"/>
+    <xacro:caster_wheel prefix="${prefix}" ns="${ns}" locationprefix="fr" locationright="1" wheel_base_dx="${mir_100_front_caster_wheel_base_dx}"/>
+    <xacro:caster_wheel prefix="${prefix}" ns="${ns}" locationprefix="bl" locationright="-1" wheel_base_dx="${mir_100_back_caster_wheel_base_dx}"/>
+    <xacro:caster_wheel prefix="${prefix}" ns="${ns}" locationprefix="br" locationright="1" wheel_base_dx="${mir_100_back_caster_wheel_base_dx}"/>
     <joint name="${prefix}base_link_surface_joint" type="fixed">
       <origin xyz="${mir_100_act_wheel_dx} 0 0.352" rpy="0 0 0" />
@@ -235,5 +236,5 @@
     <!-- set the gazebo friction parameters for the wheels -->
     <xacro:set_all_wheel_frictions prefix="${prefix}"/>
-    <xacro:p3d_base_controller prefix="${prefix}" namespace="${namespace}"/>
+    <xacro:p3d_base_controller prefix="${prefix}"/>
   </xacro:macro>
 </robot>

File: mir_description/urdf/include/sick_s300.urdf.xacro (robot description, xacro)
@@ -6,5 +6,5 @@
   <xacro:property name="laser_z" value="0.185" />
   <xacro:property name="laser_mass" value="2.0" />
-  <xacro:macro name="sick_s300" params="link topic prefix namespace">
+  <xacro:macro name="sick_s300" params="link topic prefix">
     <link name="${prefix}${link}">
       <visual>
@@ -57,6 +57,5 @@
         <plugin name="gazebo_ros_${link}_controller" filename="libgazebo_ros_ray_sensor.so">
           <ros>
-            <remapping>~/out:=${topic}</remapping>
-            <namespace>${namespace}</namespace>
+            <remapping>~/out:=${prefix}${topic}</remapping>
           </ros>
           <output_type>sensor_msgs/LaserScan</output_type>

File: mir_description/urdf/mir.urdf.xacro (robot description, xacro)
@@ -5,20 +5,16 @@
   <xacro:include filename="$(find mir_description)/urdf/include/mir_100_v1.urdf.xacro" />
   <xacro:include filename="$(find mir_description)/urdf/include/common.gazebo.xacro" />
-  <xacro:arg name="namespace" default=""/>
+  <xacro:include filename="$(find mir_description)/urdf/include/mir_100.gazebo.xacro" />
   <xacro:arg name="tf_prefix" default="" />
-  <xacro:property name="tf_prefix_val" value="$(arg tf_prefix)" />
-  <xacro:if value="${tf_prefix_val == ''}">
+  <!-- prefix can not start with a slash like a global namespace! results in TF errors -->
+  <xacro:property name="ns" value="$(arg tf_prefix)" />
+  <xacro:if value="${ns == ''}">
     <xacro:property name="prefix" value="" />
-    <xacro:property name="namespace" value=""/>
   </xacro:if>
-  <xacro:unless value="${tf_prefix_val == ''}">
-    <xacro:property name="prefix" value="${tf_prefix_val}/" />
-    <xacro:property name="namespace" value="${tf_prefix_val}"/>
+  <xacro:unless value="${ns == ''}">
+    <xacro:property name="prefix" value="${ns}/" />
   </xacro:unless>
-  <xacro:mir_100 prefix="${prefix}" namespace="${namespace}"/>
-  <!--
-  <xacro:controller_plugin_gazebo robot_namespace=""/>
-  -->
-  <xacro:diff_controller_plugin_gazebo prefix="${prefix}" namespace="${namespace}"
+  <xacro:mir_100 prefix="${prefix}" ns="${ns}"/>
+  <xacro:diff_controller_plugin_gazebo prefix="${prefix}" ns="${ns}"
     left_wheel_joint="${prefix}left_wheel_joint"
     right_wheel_joint="${prefix}right_wheel_joint"
