Commit message: Rename mir_100 -> mir
This is in preparation of mir_250 support.

File: mir_description/urdf/include/mir_v1.urdf.xacro (robot description, xacro)
@@ -3,24 +3,24 @@
   <xacro:include filename="$(find mir_description)/urdf/include/common_properties.urdf.xacro" />
   <xacro:include filename="$(find mir_description)/urdf/include/imu.gazebo.urdf.xacro" />
-  <xacro:include filename="$(find mir_description)/urdf/include/mir_100.gazebo.xacro" />
-  <xacro:include filename="$(find mir_description)/urdf/include/mir_100.transmission.xacro" />
+  <xacro:include filename="$(find mir_description)/urdf/include/mir.gazebo.xacro" />
+  <xacro:include filename="$(find mir_description)/urdf/include/mir.transmission.xacro" />
   <xacro:include filename="$(find mir_description)/urdf/include/sick_s300.urdf.xacro" />
   <xacro:property name="deg_to_rad" value="0.017453293" />
-  <xacro:property name="mir_100_base_mass" value="58.0" />
-  <xacro:property name="mir_100_act_wheel_radius" value="0.0625" />
-  <xacro:property name="mir_100_act_wheel_width" value="0.032" />
-  <xacro:property name="mir_100_act_wheel_mass" value="1.0" />
-  <xacro:property name="mir_100_act_wheel_dx" value="0.037646" />
-  <xacro:property name="mir_100_act_wheel_dy" value="0.222604" />
-  <xacro:property name="mir_100_caster_wheel_radius" value="0.0625" />
-  <xacro:property name="mir_100_caster_wheel_width" value="0.032" />
-  <xacro:property name="mir_100_caster_wheel_mass" value="1.0" />
-  <xacro:property name="mir_100_caster_wheel_dx" value="-0.0382" />
-  <xacro:property name="mir_100_caster_wheel_dy" value="0" />
-  <xacro:property name="mir_100_caster_wheel_dz" value="-0.094" />
-  <xacro:property name="mir_100_front_caster_wheel_base_dx" value="0.3037" />
-  <xacro:property name="mir_100_back_caster_wheel_base_dx"  value="0.3078" />
-  <xacro:property name="mir_100_caster_wheel_base_dy" value="0.203" />
-  <xacro:property name="mir_100_caster_wheel_base_dz" value="${mir_100_caster_wheel_radius - mir_100_caster_wheel_dz}" />
+  <xacro:property name="mir_base_mass" value="58.0" />
+  <xacro:property name="mir_act_wheel_radius" value="0.0625" />
+  <xacro:property name="mir_act_wheel_width" value="0.032" />
+  <xacro:property name="mir_act_wheel_mass" value="1.0" />
+  <xacro:property name="mir_act_wheel_dx" value="0.037646" />
+  <xacro:property name="mir_act_wheel_dy" value="0.222604" />
+  <xacro:property name="mir_caster_wheel_radius" value="0.0625" />
+  <xacro:property name="mir_caster_wheel_width" value="0.032" />
+  <xacro:property name="mir_caster_wheel_mass" value="1.0" />
+  <xacro:property name="mir_caster_wheel_dx" value="-0.0382" />
+  <xacro:property name="mir_caster_wheel_dy" value="0" />
+  <xacro:property name="mir_caster_wheel_dz" value="-0.094" />
+  <xacro:property name="mir_front_caster_wheel_base_dx" value="0.3037" />
+  <xacro:property name="mir_back_caster_wheel_base_dx"  value="0.3078" />
+  <xacro:property name="mir_caster_wheel_base_dy" value="0.203" />
+  <xacro:property name="mir_caster_wheel_base_dz" value="${mir_caster_wheel_radius - mir_caster_wheel_dz}" />
   <!-- from visually matching up the meshes of the MiR and the laser scanner -->
   <xacro:property name="laser_dx" value="0.392" />
@@ -29,5 +29,5 @@
   <xacro:macro name="actuated_wheel" params="prefix locationprefix locationright">
     <joint name="${prefix}${locationprefix}_wheel_joint" type="continuous">
-      <origin xyz="0.0 ${-mir_100_act_wheel_dy * locationright} ${mir_100_act_wheel_radius}" rpy="0 0 0" />
+      <origin xyz="0.0 ${-mir_act_wheel_dy * locationright} ${mir_act_wheel_radius}" rpy="0 0 0" />
       <parent link="${prefix}base_link" />
       <child link="${prefix}${locationprefix}_wheel_link" />
@@ -36,5 +36,5 @@
     </joint>
     <link name="${prefix}${locationprefix}_wheel_link">
-      <xacro:cylinder_inertial mass="${mir_100_act_wheel_mass}" radius="${mir_100_act_wheel_radius}" length="${mir_100_act_wheel_width}">
+      <xacro:cylinder_inertial mass="${mir_act_wheel_mass}" radius="${mir_act_wheel_radius}" length="${mir_act_wheel_width}">
         <origin xyz="0 0 0" rpy="${0.5 * pi} 0 0" />
       </xacro:cylinder_inertial>
@@ -42,5 +42,5 @@
         <origin xyz="0 0 0" rpy="${pi/2} 0 0" />
         <geometry>
-          <cylinder radius="${mir_100_act_wheel_radius}" length="${mir_100_act_wheel_width}" />
+          <cylinder radius="${mir_act_wheel_radius}" length="${mir_act_wheel_width}" />
         </geometry>
         <xacro:insert_block name="material_dark_grey" />
@@ -49,5 +49,5 @@
         <origin xyz="0 0 0" rpy="${pi/2} 0 0" />
         <geometry>
-          <cylinder radius="${mir_100_act_wheel_radius}" length="${mir_100_act_wheel_width}" />
+          <cylinder radius="${mir_act_wheel_radius}" length="${mir_act_wheel_width}" />
         </geometry>
       </collision>
@@ -60,5 +60,5 @@
     <!-- caster hub -->
     <joint name="${prefix}${locationprefix}_caster_rotation_joint" type="continuous">
-      <origin xyz="${wheel_base_dx} ${-mir_100_caster_wheel_base_dy * locationright} ${mir_100_caster_wheel_base_dz}" rpy="0 0 0" />
+      <origin xyz="${wheel_base_dx} ${-mir_caster_wheel_base_dy * locationright} ${mir_caster_wheel_base_dz}" rpy="0 0 0" />
       <parent link="${prefix}base_link" />
       <child link="${prefix}${locationprefix}_caster_rotation_link" />
@@ -98,5 +98,5 @@
     <!-- caster wheel -->
     <joint name="${prefix}${locationprefix}_caster_wheel_joint" type="continuous">
-      <origin xyz="${mir_100_caster_wheel_dx} ${-mir_100_caster_wheel_dy * locationright} ${mir_100_caster_wheel_dz}" rpy="0 0 0" />
+      <origin xyz="${mir_caster_wheel_dx} ${-mir_caster_wheel_dy * locationright} ${mir_caster_wheel_dz}" rpy="0 0 0" />
       <parent link="${prefix}${locationprefix}_caster_rotation_link" />
       <child link="${prefix}${locationprefix}_caster_wheel_link" />
@@ -104,5 +104,5 @@
     </joint>
     <link name="${prefix}${locationprefix}_caster_wheel_link">
-      <xacro:cylinder_inertial mass="${mir_100_caster_wheel_mass}" radius="${mir_100_caster_wheel_radius}" length="${mir_100_caster_wheel_width}">
+      <xacro:cylinder_inertial mass="${mir_caster_wheel_mass}" radius="${mir_caster_wheel_radius}" length="${mir_caster_wheel_width}">
         <origin xyz="0 0 0" rpy="${0.5 * pi} 0 0" />
       </xacro:cylinder_inertial>
@@ -110,5 +110,5 @@
         <origin xyz="0 0 0" rpy="${pi/2} 0 0" />
         <geometry>
-          <cylinder radius="${mir_100_caster_wheel_radius}" length="${mir_100_caster_wheel_width}" />
+          <cylinder radius="${mir_caster_wheel_radius}" length="${mir_caster_wheel_width}" />
         </geometry>
         <xacro:insert_block name="material_dark_grey" />
@@ -117,5 +117,5 @@
         <origin xyz="0 0 0" rpy="${pi/2} 0 0" />
         <geometry>
-          <cylinder radius="${mir_100_caster_wheel_radius}" length="${mir_100_caster_wheel_width}" />
+          <cylinder radius="${mir_caster_wheel_radius}" length="${mir_caster_wheel_width}" />
         </geometry>
       </collision>
@@ -125,5 +125,5 @@
     </gazebo>
   </xacro:macro>
-  <xacro:macro name="mir_100" params="prefix">
+  <xacro:macro name="mir" params="prefix">
     <link name="${prefix}base_footprint" />
     <joint name="${prefix}base_joint" type="fixed">
@@ -133,9 +133,9 @@
     </joint>
     <link name="${prefix}base_link">
-      <xacro:box_inertial mass="${mir_100_base_mass}" x="0.9" y="0.58" z="0.3">
-        <origin xyz="${mir_100_act_wheel_dx} 0 0.20" rpy="0 0 0" />
+      <xacro:box_inertial mass="${mir_base_mass}" x="0.9" y="0.58" z="0.3">
+        <origin xyz="${mir_act_wheel_dx} 0 0.20" rpy="0 0 0" />
       </xacro:box_inertial>
       <visual>
-        <origin xyz="${mir_100_act_wheel_dx} 0 0" rpy="0 0 0" />
+        <origin xyz="${mir_act_wheel_dx} 0 0" rpy="0 0 0" />
         <geometry>
           <mesh filename="package://mir_description/meshes/visual/mir_100_base.stl" />
@@ -144,5 +144,5 @@
       </visual>
       <collision>
-        <origin xyz="${mir_100_act_wheel_dx} 0 0" rpy="0 0 0" />
+        <origin xyz="${mir_act_wheel_dx} 0 0" rpy="0 0 0" />
         <geometry>
           <mesh filename="package://mir_description/meshes/collision/mir_100_base.stl" />
@@ -174,5 +174,5 @@
       <parent link="${prefix}base_link" />
       <child link="${prefix}front_laser_link" />
-      <origin xyz="${laser_dx + mir_100_act_wheel_dx} ${laser_dy} ${laser_dz}" rpy="0.0 0.0 ${0.25 * pi}" />
+      <origin xyz="${laser_dx + mir_act_wheel_dx} ${laser_dy} ${laser_dz}" rpy="0.0 0.0 ${0.25 * pi}" />
     </joint>
     <xacro:sick_s300 prefix="${prefix}" link="front_laser_link" topic="f_scan" />
@@ -180,5 +180,5 @@
       <parent link="${prefix}base_link" />
       <child link="${prefix}back_laser_link" />
-      <origin xyz="${-laser_dx + mir_100_act_wheel_dx} ${-laser_dy} ${laser_dz}" rpy="0.0 0.0 ${-0.75 * pi}" />
+      <origin xyz="${-laser_dx + mir_act_wheel_dx} ${-laser_dy} ${laser_dz}" rpy="0.0 0.0 ${-0.75 * pi}" />
     </joint>
     <xacro:sick_s300 prefix="${prefix}" link="back_laser_link" topic="b_scan" />
@@ -199,10 +199,10 @@
     <xacro:actuated_wheel prefix="${prefix}" locationprefix="left" locationright="-1"/>
     <xacro:actuated_wheel prefix="${prefix}" locationprefix="right" locationright="1"/>
-    <xacro:caster_wheel prefix="${prefix}" locationprefix="fl" locationright="-1" wheel_base_dx="${mir_100_front_caster_wheel_base_dx + mir_100_act_wheel_dx}"/>
-    <xacro:caster_wheel prefix="${prefix}" locationprefix="fr" locationright="1" wheel_base_dx="${mir_100_front_caster_wheel_base_dx + mir_100_act_wheel_dx}"/>
-    <xacro:caster_wheel prefix="${prefix}" locationprefix="bl" locationright="-1" wheel_base_dx="${-mir_100_back_caster_wheel_base_dx + mir_100_act_wheel_dx}"/>
-    <xacro:caster_wheel prefix="${prefix}" locationprefix="br" locationright="1" wheel_base_dx="${-mir_100_back_caster_wheel_base_dx + mir_100_act_wheel_dx}"/>
+    <xacro:caster_wheel prefix="${prefix}" locationprefix="fl" locationright="-1" wheel_base_dx="${mir_front_caster_wheel_base_dx + mir_act_wheel_dx}"/>
+    <xacro:caster_wheel prefix="${prefix}" locationprefix="fr" locationright="1" wheel_base_dx="${mir_front_caster_wheel_base_dx + mir_act_wheel_dx}"/>
+    <xacro:caster_wheel prefix="${prefix}" locationprefix="bl" locationright="-1" wheel_base_dx="${-mir_back_caster_wheel_base_dx + mir_act_wheel_dx}"/>
+    <xacro:caster_wheel prefix="${prefix}" locationprefix="br" locationright="1" wheel_base_dx="${-mir_back_caster_wheel_base_dx + mir_act_wheel_dx}"/>
     <joint name="${prefix}base_link_surface_joint" type="fixed">
-      <origin xyz="${mir_100_act_wheel_dx} 0 0.352" rpy="0 0 0" />
+      <origin xyz="${mir_act_wheel_dx} 0 0.352" rpy="0 0 0" />
       <parent link="${prefix}base_link" />
       <child link="${prefix}surface" />
@@ -210,5 +210,5 @@
     </joint>
     <link name="${prefix}surface"/>
-    <xacro:mir_100_wheel_transmissions prefix="${prefix}"/>
+    <xacro:mir_wheel_transmissions prefix="${prefix}"/>
     <!-- set the gazebo friction parameters for the wheels -->
     <xacro:set_all_wheel_frictions prefix="${prefix}"/>

File: mir_description/urdf/mir.urdf.xacro (robot description, xacro)
@@ -1,7 +1,7 @@
 <?xml version="1.0"?>
 <robot xmlns:xacro="http://ros.org/wiki/xacro"
-       name="mir_100" >
-  <!-- MiR100 base -->
-  <xacro:include filename="$(find mir_description)/urdf/include/mir_100_v1.urdf.xacro" />
+       name="mir" >
+  <!-- MiR base -->
+  <xacro:include filename="$(find mir_description)/urdf/include/mir_v1.urdf.xacro" />
   <xacro:include filename="$(find mir_description)/urdf/include/common.gazebo.xacro" />
   <xacro:arg name="tf_prefix" default="" />
@@ -13,5 +13,5 @@
     <xacro:property name="prefix" value="${tf_prefix_}/" />
   </xacro:unless>
-  <xacro:mir_100 prefix="${prefix}"/>
+  <xacro:mir prefix="${prefix}"/>
   <xacro:controller_plugin_gazebo robot_namespace=""/>
   <!-- instead of the controller_plugin_gazebo, you can use the diffdrive controller like this:
@@ -19,6 +19,6 @@
       left_wheel_joint="left_wheel_joint"
       right_wheel_joint="right_wheel_joint"
-      wheel_separation="${2*mir_100_act_wheel_dy}"
-      wheel_radius="${mir_100_act_wheel_radius}"/>
+      wheel_separation="${2*mir_act_wheel_dy}"
+      wheel_radius="${mir_act_wheel_radius}"/>
   -->
 </robot>

Commit message: URDF: Make wheels black
This increases the contrast for the MiR 250 robot.

File: mir_description/urdf/include/mir_v1.urdf.xacro (robot description, xacro)
@@ -44,5 +44,5 @@
           <cylinder radius="${mir_act_wheel_radius}" length="${mir_act_wheel_width}" />
         </geometry>
-        <xacro:insert_block name="material_dark_grey" />
+        <xacro:insert_block name="material_black" />
       </visual>
       <collision>
@@ -54,5 +54,5 @@
     </link>
     <gazebo reference="${prefix}${locationprefix}_wheel_link">
-      <material>Gazebo/DarkGrey</material>
+      <material>Gazebo/FlatBlack</material>
     </gazebo>
   </xacro:macro>
@@ -112,5 +112,5 @@
           <cylinder radius="${mir_caster_wheel_radius}" length="${mir_caster_wheel_width}" />
         </geometry>
-        <xacro:insert_block name="material_dark_grey" />
+        <xacro:insert_block name="material_black" />
       </visual>
       <collision>
@@ -122,5 +122,5 @@
     </link>
     <gazebo reference="${prefix}${locationprefix}_caster_wheel_link">
-      <material>Gazebo/DarkGrey</material>
+      <material>Gazebo/FlatBlack</material>
     </gazebo>
   </xacro:macro>

Commit message: Add arg mir_type to launch files and urdfs

File: mir_description/urdf/include/mir_v1.urdf.xacro (robot description, xacro)
@@ -1,4 +1,6 @@
 <?xml version="1.0"?>
 <robot xmlns:xacro="http://ros.org/wiki/xacro">
+  <xacro:arg name="mir_type" default="mir_100" />      <!-- The MiR variant. Can be "mir_100" or "mir_250" for now.-->
+  <xacro:property name="mir_type" value="$(arg mir_type)" />  <!-- necessary because args cannot be accessed inside ${} expressions -->
   <xacro:include filename="$(find mir_description)/urdf/include/common_properties.urdf.xacro" />
   <xacro:include filename="$(find mir_description)/urdf/include/imu.gazebo.urdf.xacro" />
@@ -125,5 +127,5 @@
     </gazebo>
   </xacro:macro>
-  <xacro:macro name="mir" params="prefix">
+  <xacro:macro name="mir" params="mir_type prefix">
     <link name="${prefix}base_footprint" />
     <joint name="${prefix}base_joint" type="fixed">
@@ -139,5 +141,5 @@
         <origin xyz="${mir_act_wheel_dx} 0 0" rpy="0 0 0" />
         <geometry>
-          <mesh filename="package://mir_description/meshes/visual/mir_100_base.stl" />
+          <mesh filename="package://mir_description/meshes/visual/${mir_type}_base.stl" />
         </geometry>
         <xacro:insert_block name="material_white" />
@@ -146,5 +148,5 @@
         <origin xyz="${mir_act_wheel_dx} 0 0" rpy="0 0 0" />
         <geometry>
-          <mesh filename="package://mir_description/meshes/collision/mir_100_base.stl" />
+          <mesh filename="package://mir_description/meshes/collision/${mir_type}_base.stl" />
         </geometry>
       </collision>

File: mir_description/urdf/mir.urdf.xacro (robot description, xacro)
@@ -13,5 +13,5 @@
     <xacro:property name="prefix" value="${tf_prefix_}/" />
   </xacro:unless>
-  <xacro:mir prefix="${prefix}"/>
+  <xacro:mir prefix="${prefix}" />
   <xacro:controller_plugin_gazebo robot_namespace=""/>
   <!-- instead of the controller_plugin_gazebo, you can use the diffdrive controller like this:

Commit message: URDF: Add mir_250

File: mir_description/urdf/include/mir_v1.urdf.xacro (robot description, xacro)
@@ -10,9 +10,18 @@
   <xacro:property name="deg_to_rad" value="0.017453293" />
   <xacro:property name="mir_base_mass" value="58.0" />
-  <xacro:property name="mir_act_wheel_radius" value="0.0625" />
-  <xacro:property name="mir_act_wheel_width" value="0.032" />
-  <xacro:property name="mir_act_wheel_mass" value="1.0" />
-  <xacro:property name="mir_act_wheel_dx" value="0.037646" />
-  <xacro:property name="mir_act_wheel_dy" value="0.222604" />
+  <xacro:if value="${mir_type == 'mir_100'}">
+    <xacro:property name="mir_act_wheel_radius" value="0.0625" />
+    <xacro:property name="mir_act_wheel_width" value="0.032" />
+    <xacro:property name="mir_act_wheel_mass" value="1.0" />
+    <xacro:property name="mir_act_wheel_dx" value="0.037646" />
+    <xacro:property name="mir_act_wheel_dy" value="0.222604" />
+  </xacro:if>
+  <xacro:if value="${mir_type == 'mir_250'}">
+    <xacro:property name="mir_act_wheel_radius" value="0.100" />
+    <xacro:property name="mir_act_wheel_width" value="0.038" />
+    <xacro:property name="mir_act_wheel_mass" value="1.0" />
+    <xacro:property name="mir_act_wheel_dx" value="-0.004485" />
+    <xacro:property name="mir_act_wheel_dy" value="0.2015" />
+  </xacro:if>
   <xacro:property name="mir_caster_wheel_radius" value="0.0625" />
   <xacro:property name="mir_caster_wheel_width" value="0.032" />
@@ -22,10 +31,22 @@
   <xacro:property name="mir_caster_wheel_dz" value="-0.094" />
   <xacro:property name="mir_front_caster_wheel_base_dx" value="0.3037" />
-  <xacro:property name="mir_back_caster_wheel_base_dx"  value="0.3078" />
-  <xacro:property name="mir_caster_wheel_base_dy" value="0.203" />
+  <xacro:if value="${mir_type == 'mir_100'}">
+    <xacro:property name="mir_back_caster_wheel_base_dx"  value="0.3078" />
+    <xacro:property name="mir_caster_wheel_base_dy" value="0.203" />
+  </xacro:if>
+  <xacro:if value="${mir_type == 'mir_250'}">
+    <xacro:property name="mir_back_caster_wheel_base_dx"  value="0.296" />
+    <xacro:property name="mir_caster_wheel_base_dy" value="0.188" />
+  </xacro:if>
   <xacro:property name="mir_caster_wheel_base_dz" value="${mir_caster_wheel_radius - mir_caster_wheel_dz}" />
   <!-- from visually matching up the meshes of the MiR and the laser scanner -->
-  <xacro:property name="laser_dx" value="0.392" />
-  <xacro:property name="laser_dy" value="0.2358" />
+  <xacro:if value="${mir_type == 'mir_100'}">
+    <xacro:property name="laser_dx" value="0.392" />
+    <xacro:property name="laser_dy" value="0.2358" />
+  </xacro:if>
+  <xacro:if value="${mir_type == 'mir_250'}">
+    <xacro:property name="laser_dx" value="0.315" />
+    <xacro:property name="laser_dy" value="0.205" />
+  </xacro:if>
   <xacro:property name="laser_dz" value="0.1914" />
   <xacro:macro name="actuated_wheel" params="prefix locationprefix locationright">
@@ -86,5 +107,10 @@
           <mesh filename="package://mir_description/meshes/visual/caster_wheel_base.stl" />
         </geometry>
-        <xacro:insert_block name="material_silver" />
+        <xacro:if value="${mir_type == 'mir_100'}">
+          <xacro:insert_block name="material_silver" />
+        </xacro:if>
+        <xacro:if value="${mir_type == 'mir_250'}">
+          <xacro:insert_block name="material_black" />
+        </xacro:if>
       </visual>
       <collision>
@@ -96,5 +122,10 @@
     </link>
     <gazebo reference="${prefix}${locationprefix}_caster_rotation_link">
-      <material>Gazebo/Grey</material>
+      <xacro:if value="${mir_type == 'mir_100'}">
+        <material>Gazebo/Grey</material>
+      </xacro:if>
+      <xacro:if value="${mir_type == 'mir_250'}">
+        <material>Gazebo/FlatBlack</material>
+      </xacro:if>
     </gazebo>
     <!-- caster wheel -->
@@ -127,5 +158,5 @@
     </gazebo>
   </xacro:macro>
-  <xacro:macro name="mir" params="mir_type prefix">
+  <xacro:macro name="mir" params="prefix">
     <link name="${prefix}base_footprint" />
     <joint name="${prefix}base_joint" type="fixed">
@@ -143,5 +174,10 @@
           <mesh filename="package://mir_description/meshes/visual/${mir_type}_base.stl" />
         </geometry>
-        <xacro:insert_block name="material_white" />
+        <xacro:if value="${mir_type == 'mir_100'}">
+          <xacro:insert_block name="material_white" />
+        </xacro:if>
+        <xacro:if value="${mir_type == 'mir_250'}">
+          <xacro:insert_block name="material_dark_grey" />
+        </xacro:if>
       </visual>
       <collision>
@@ -153,5 +189,10 @@
     </link>
     <gazebo reference="${prefix}base_link">
-      <material>Gazebo/White</material>
+      <xacro:if value="${mir_type == 'mir_100'}">
+        <material>Gazebo/White</material>
+      </xacro:if>
+      <xacro:if value="${mir_type == 'mir_250'}">
+        <material>Gazebo/DarkGrey</material>
+      </xacro:if>
     </gazebo>
     <!-- IMU -->

Commit message: URDF: Update masses according to data sheet

File: mir_description/urdf/include/mir_v1.urdf.xacro (robot description, xacro)
@@ -9,6 +9,6 @@
   <xacro:include filename="$(find mir_description)/urdf/include/sick_s300.urdf.xacro" />
   <xacro:property name="deg_to_rad" value="0.017453293" />
-  <xacro:property name="mir_base_mass" value="58.0" />
   <xacro:if value="${mir_type == 'mir_100'}">
+    <xacro:property name="mir_base_mass" value="77.0" />
     <xacro:property name="mir_act_wheel_radius" value="0.0625" />
     <xacro:property name="mir_act_wheel_width" value="0.032" />
@@ -18,4 +18,5 @@
   </xacro:if>
   <xacro:if value="${mir_type == 'mir_250'}">
+    <xacro:property name="mir_base_mass" value="97.0" />
     <xacro:property name="mir_act_wheel_radius" value="0.100" />
     <xacro:property name="mir_act_wheel_width" value="0.038" />

Commit message: URDF: Pull out inertia properties

File: mir_description/urdf/include/mir_v1.urdf.xacro (robot description, xacro)
@@ -9,4 +9,10 @@
   <xacro:include filename="$(find mir_description)/urdf/include/sick_s300.urdf.xacro" />
   <xacro:property name="deg_to_rad" value="0.017453293" />
+  <xacro:property name="mir_base_inertial_x" value="0.0" />
+  <xacro:property name="mir_base_inertial_y" value="0.0" />
+  <xacro:property name="mir_base_inertial_z" value="0.20" />
+  <xacro:property name="mir_base_inertial_x_length" value="0.9" />
+  <xacro:property name="mir_base_inertial_y_length" value="0.58" />
+  <xacro:property name="mir_base_inertial_z_length" value="0.3" />
   <xacro:if value="${mir_type == 'mir_100'}">
     <xacro:property name="mir_base_mass" value="77.0" />
@@ -167,6 +173,6 @@
     </joint>
     <link name="${prefix}base_link">
-      <xacro:box_inertial mass="${mir_base_mass}" x="0.9" y="0.58" z="0.3">
-        <origin xyz="${mir_act_wheel_dx} 0 0.20" rpy="0 0 0" />
+      <xacro:box_inertial mass="${mir_base_mass}" x="${mir_base_inertial_x_length}" y="${mir_base_inertial_y_length}" z="${mir_base_inertial_z_length}">
+        <origin xyz="${mir_base_inertial_x + mir_act_wheel_dx} ${mir_base_inertial_y} ${mir_base_inertial_z}" rpy="0 0 0" />
       </xacro:box_inertial>
       <visual>
