Commit message: Add TFs for ultrasound sensors

File: mir_description/urdf/include/mir_100_v1.urdf.xacro (robot description, xacro)
@@ -180,4 +180,17 @@
     </joint>
     <xacro:sick_s300 link="${prefix}back_laser_link" topic="b_scan" />
+    <!-- Ultrasound sensors -->
+    <joint name="${prefix}us_1_joint" type="fixed">   <!-- right ultrasound -->
+      <parent link="${prefix}base_link" />
+      <child link="${prefix}us_1_frame" />
+      <origin xyz="0.45 -0.12 0.16 " rpy="0 0 0" />  <!-- from visually matching to the mesh of the MiR -->
+    </joint>
+    <link name="${prefix}us_1_frame" />
+    <joint name="${prefix}us_2_joint" type="fixed">   <!-- left ultrasound -->
+      <parent link="${prefix}base_link" />
+      <child link="${prefix}us_2_frame" />
+      <origin xyz="0.45 0.12 0.16 " rpy="0 0 0" />  <!-- from visually matching to the mesh of the MiR -->
+    </joint>
+    <link name="${prefix}us_2_frame" />
     <!-- wheels -->
     <xacro:actuated_wheel prefix="${prefix}" locationprefix="left" locationright="-1"/>

Commit message: added virtual laserscan link

File: mir_description/urdf/include/mir_100_v1.urdf.xacro (robot description, xacro)
@@ -185,4 +185,12 @@
     <link name="${prefix}imu_frame" />
     <!-- Laser scanners -->
+    <!-- virtual link for merged laserscan-->
+    <joint name="${prefix}base_link_to_virtual_laser_joint" type="fixed">
+      <parent link="${prefix}base_link" />
+      <child link="${prefix}virtual_laser_link" />
+      <origin xyz="0.0 0.0 0.1914" rpy="0.0 0.0 0" />
+    </joint>
+    <link name="${prefix}virtual_laser_link">
+    </link>
     <joint name="${prefix}base_link_to_front_laser_joint" type="fixed">
       <parent link="${prefix}base_link" />

Commit message: hotfix virtual laser link scan_merger

File: mir_description/urdf/include/mir_100_v1.urdf.xacro (robot description, xacro)
@@ -189,5 +189,5 @@
       <parent link="${prefix}base_link" />
       <child link="${prefix}virtual_laser_link" />
-      <origin xyz="0.0 0.0 0.1914" rpy="0.0 0.0 0" />
+      <origin xyz="0.0 0.0 0.25" rpy="0.0 0.0 0" />
     </joint>
     <link name="${prefix}virtual_laser_link">

Commit message: Use cylinders instead of STLs for wheel collision geometries
When using the STL meshes, there were lots of inconsistent contacts
between the wheels and the ground. This resulted in lots of small
"vibrations" of the robot due to unstable repulsive forces between
ground and wheels, which were measured by the simulated IMU. Using
cylinders as collision geometries fixes that.

Fixes #99.

File: mir_description/urdf/include/mir_100_v1.urdf.xacro (robot description, xacro)
@@ -44,7 +44,7 @@
       </visual>
       <collision>
-        <origin xyz="0 0 0" rpy="0 0 0" />
-        <geometry>
-          <mesh filename="package://mir_description/meshes/visual/wheel.stl" />
+        <origin xyz="0 0 0" rpy="${pi/2} 0 0" />
+        <geometry>
+          <cylinder radius="${mir_100_act_wheel_radius}" length="${mir_100_act_wheel_width}" />
         </geometry>
       </collision>
@@ -112,7 +112,7 @@
       </visual>
       <collision>
-        <origin xyz="0 0 0" rpy="0 0 0" />
-        <geometry>
-          <mesh filename="package://mir_description/meshes/visual/wheel.stl" />
+        <origin xyz="0 0 0" rpy="${pi/2} 0 0" />
+        <geometry>
+          <cylinder radius="${mir_100_caster_wheel_radius}" length="${mir_100_caster_wheel_width}" />
         </geometry>
       </collision>

Commit message: Replace gazebo_plugins IMU with hector_gazebo_plugins
The gazebo_plugins IMU has a very bad noise model (same stdev for
everything). The IMU plugin from hector_gazebo_plugins is much better.

See #99.

File: mir_description/urdf/include/mir_100_v1.urdf.xacro (robot description, xacro)
@@ -23,5 +23,4 @@
   <xacro:property name="mir_100_caster_wheel_base_dy" value="0.203" />
   <xacro:property name="mir_100_caster_wheel_base_dz" value="${mir_100_caster_wheel_radius-mir_100_caster_wheel_dz}" />
-  <xacro:property name="imu_stdev" value="0.00017" />
   <xacro:macro name="actuated_wheel" params="prefix locationprefix locationright">
     <joint name="${prefix}${locationprefix}_wheel_joint" type="continuous">
@@ -157,5 +156,5 @@
     </joint>
     <link name="${prefix}imu_link" />
-    <xacro:imu_gazebo link="${prefix}imu_link" imu_topic="imu_data" update_rate="50.0" stdev="${imu_stdev}" />
+    <xacro:imu_gazebo link="${prefix}imu_link" imu_topic="imu_data" update_rate="50.0" />
     <!-- Create an alias for imu_link. This is necessary because the real MiR's
          TF has imu_link, but the imu_data topic is published in the imu_frame

Commit message: Refactor URDF to prepare for MiR250 support
* specify caster wheel dx, radius and width independent of active wheel
* use cylinder geometric primitive instead of mesh for visual tag of wheels
* pull out laser positions into properties

File: mir_description/urdf/include/mir_100_v1.urdf.xacro (robot description, xacro)
@@ -13,14 +13,18 @@
   <xacro:property name="mir_100_act_wheel_dx" value="0.037646" />
   <xacro:property name="mir_100_act_wheel_dy" value="0.222604" />
-  <xacro:property name="mir_100_caster_wheel_radius" value="${mir_100_act_wheel_radius}" />
-  <xacro:property name="mir_100_caster_wheel_width" value="${mir_100_act_wheel_width}" />
-  <xacro:property name="mir_100_caster_wheel_mass" value="${mir_100_act_wheel_mass}" />
+  <xacro:property name="mir_100_caster_wheel_radius" value="0.0625" />
+  <xacro:property name="mir_100_caster_wheel_width" value="0.032" />
+  <xacro:property name="mir_100_caster_wheel_mass" value="1.0" />
   <xacro:property name="mir_100_caster_wheel_dx" value="-0.0382" />
   <xacro:property name="mir_100_caster_wheel_dy" value="0" />
   <xacro:property name="mir_100_caster_wheel_dz" value="-0.094" />
-  <xacro:property name="mir_100_front_caster_wheel_base_dx" value="0.341346" />
-  <xacro:property name="mir_100_back_caster_wheel_base_dx" value="-0.270154" />
+  <xacro:property name="mir_100_front_caster_wheel_base_dx" value="0.3037" />
+  <xacro:property name="mir_100_back_caster_wheel_base_dx"  value="0.3078" />
   <xacro:property name="mir_100_caster_wheel_base_dy" value="0.203" />
-  <xacro:property name="mir_100_caster_wheel_base_dz" value="${mir_100_caster_wheel_radius-mir_100_caster_wheel_dz}" />
+  <xacro:property name="mir_100_caster_wheel_base_dz" value="${mir_100_caster_wheel_radius - mir_100_caster_wheel_dz}" />
+  <!-- from visually matching up the meshes of the MiR and the laser scanner -->
+  <xacro:property name="laser_dx" value="0.392" />
+  <xacro:property name="laser_dy" value="0.2358" />
+  <xacro:property name="laser_dz" value="0.1914" />
   <xacro:macro name="actuated_wheel" params="prefix locationprefix locationright">
     <joint name="${prefix}${locationprefix}_wheel_joint" type="continuous">
@@ -36,7 +40,7 @@
       </xacro:cylinder_inertial>
       <visual>
-        <origin xyz="0 0 0" rpy="0 0 0" />
-        <geometry>
-          <mesh filename="package://mir_description/meshes/visual/wheel.stl" />
+        <origin xyz="0 0 0" rpy="${pi/2} 0 0" />
+        <geometry>
+          <cylinder radius="${mir_100_act_wheel_radius}" length="${mir_100_act_wheel_width}" />
         </geometry>
         <xacro:insert_block name="material_dark_grey" />
@@ -104,7 +108,7 @@
       </xacro:cylinder_inertial>
       <visual>
-        <origin xyz="0 0 0" rpy="0 0 0" />
-        <geometry>
-          <mesh filename="package://mir_description/meshes/visual/wheel.stl" />
+        <origin xyz="0 0 0" rpy="${pi/2} 0 0" />
+        <geometry>
+          <cylinder radius="${mir_100_caster_wheel_radius}" length="${mir_100_caster_wheel_width}" />
         </geometry>
         <xacro:insert_block name="material_dark_grey" />
@@ -170,5 +174,5 @@
       <parent link="${prefix}base_link" />
       <child link="${prefix}front_laser_link" />
-      <origin xyz="0.4288 0.2358 0.1914" rpy="0.0 0.0 ${0.25 * pi}" />  <!-- from visually matching up the meshes of the MiR and the laser scanner -->
+      <origin xyz="${laser_dx + mir_100_act_wheel_dx} ${laser_dy} ${laser_dz}" rpy="0.0 0.0 ${0.25 * pi}" />
     </joint>
     <xacro:sick_s300 prefix="${prefix}" link="front_laser_link" topic="f_scan" />
@@ -176,5 +180,5 @@
       <parent link="${prefix}base_link" />
       <child link="${prefix}back_laser_link" />
-      <origin xyz="-0.3548 -0.2352 0.1914" rpy="0.0 0.0 ${-0.75 * pi}" />  <!-- from visually matching up the meshes of the MiR and the laser scanner -->
+      <origin xyz="${-laser_dx + mir_100_act_wheel_dx} ${-laser_dy} ${laser_dz}" rpy="0.0 0.0 ${-0.75 * pi}" />
     </joint>
     <xacro:sick_s300 prefix="${prefix}" link="back_laser_link" topic="b_scan" />
@@ -195,8 +199,8 @@
     <xacro:actuated_wheel prefix="${prefix}" locationprefix="left" locationright="-1"/>
     <xacro:actuated_wheel prefix="${prefix}" locationprefix="right" locationright="1"/>
-    <xacro:caster_wheel prefix="${prefix}" locationprefix="fl" locationright="-1" wheel_base_dx="${mir_100_front_caster_wheel_base_dx}"/>
-    <xacro:caster_wheel prefix="${prefix}" locationprefix="fr" locationright="1" wheel_base_dx="${mir_100_front_caster_wheel_base_dx}"/>
-    <xacro:caster_wheel prefix="${prefix}" locationprefix="bl" locationright="-1" wheel_base_dx="${mir_100_back_caster_wheel_base_dx}"/>
-    <xacro:caster_wheel prefix="${prefix}" locationprefix="br" locationright="1" wheel_base_dx="${mir_100_back_caster_wheel_base_dx}"/>
+    <xacro:caster_wheel prefix="${prefix}" locationprefix="fl" locationright="-1" wheel_base_dx="${mir_100_front_caster_wheel_base_dx + mir_100_act_wheel_dx}"/>
+    <xacro:caster_wheel prefix="${prefix}" locationprefix="fr" locationright="1" wheel_base_dx="${mir_100_front_caster_wheel_base_dx + mir_100_act_wheel_dx}"/>
+    <xacro:caster_wheel prefix="${prefix}" locationprefix="bl" locationright="-1" wheel_base_dx="${-mir_100_back_caster_wheel_base_dx + mir_100_act_wheel_dx}"/>
+    <xacro:caster_wheel prefix="${prefix}" locationprefix="br" locationright="1" wheel_base_dx="${-mir_100_back_caster_wheel_base_dx + mir_100_act_wheel_dx}"/>
     <joint name="${prefix}base_link_surface_joint" type="fixed">
       <origin xyz="${mir_100_act_wheel_dx} 0 0.352" rpy="0 0 0" />

Commit message: fix robot tilting + laser scans drifting

File: mir_description/urdf/include/mir_100_v1.urdf.xacro (robot description, xacro)
@@ -46,5 +46,5 @@
         <origin xyz="0 0 0" rpy="0 0 0" />
         <geometry>
-          <mesh filename="package://mir_description/meshes/visual/wheel.stl" />
+          <cylinder radius="${mir_100_act_wheel_radius}" length="${mir_100_act_wheel_width}" />
         </geometry>
       </collision>
@@ -95,5 +95,5 @@
         <origin xyz="0 0 0" rpy="0 0 0" />
         <geometry>
-          <mesh filename="package://mir_description/meshes/collision/caster_wheel_base.stl" />
+          <cylinder radius="${mir_100_caster_wheel_radius}" length="${mir_100_caster_wheel_width}" />
         </geometry>
       </collision>

Commit message: Revert "fix robot tilting + laser scans drifting"
This reverts commit 39d13c9c48e0282fe732a15fb8d8cb49edc3ceca.

File: mir_description/urdf/include/mir_100_v1.urdf.xacro (robot description, xacro)
@@ -46,5 +46,5 @@
         <origin xyz="0 0 0" rpy="0 0 0" />
         <geometry>
-          <cylinder radius="${mir_100_act_wheel_radius}" length="${mir_100_act_wheel_width}" />
+          <mesh filename="package://mir_description/meshes/visual/wheel.stl" />
         </geometry>
       </collision>
@@ -95,5 +95,5 @@
         <origin xyz="0 0 0" rpy="0 0 0" />
         <geometry>
-          <cylinder radius="${mir_100_caster_wheel_radius}" length="${mir_100_caster_wheel_width}" />
+          <mesh filename="package://mir_description/meshes/collision/caster_wheel_base.stl" />
         </geometry>
       </collision>

Commit message: recherry-picking 063d4e7

File: mir_description/urdf/include/mir_100_v1.urdf.xacro (robot description, xacro)
@@ -44,7 +44,7 @@
       </visual>
       <collision>
-        <origin xyz="0 0 0" rpy="0 0 0" />
-        <geometry>
-          <mesh filename="package://mir_description/meshes/visual/wheel.stl" />
+        <origin xyz="0 0 0" rpy="${pi/2} 0 0" />
+        <geometry>
+          <cylinder radius="${mir_100_act_wheel_radius}" length="${mir_100_act_wheel_width}" />
         </geometry>
       </collision>
@@ -130,7 +130,7 @@
       </visual>
       <collision>
-        <origin xyz="0 0 0" rpy="0 0 0" />
-        <geometry>
-          <mesh filename="package://mir_description/meshes/visual/wheel.stl" />
+        <origin xyz="0 0 0" rpy="${pi/2} 0 0" />
+        <geometry>
+          <cylinder radius="${mir_100_caster_wheel_radius}" length="${mir_100_caster_wheel_width}" />
         </geometry>
       </collision>
