Commit message: 26 tune wheel friction and damping parameters simulation (#27)
* separated wheel parts to simplify urdf build

* Changed MiR100 mass to 78.2kg

* allow urdf to parse collision parameters for gazbeo

* cherry-picked intertia from 91952d8

* applied torsional force, updated contact collisons

* tuned wheel frictions and contacs more

File: mir_description/urdf/include/mir_100.gazebo.xacro (robot description, xacro)
@@ -35,21 +35,4 @@
     </gazebo>
   </xacro:macro>
-  <xacro:macro name="set_wheel_friction" params="link friction">
-    <gazebo reference="${link}">
-      <mu1 value="${friction}"/>
-      <mu2 value="${friction}"/>
-      <kp value="10000000.0"/>
-      <kd value="1.0"/>
-      <minDepth>0.01</minDepth>
-    </gazebo>
-  </xacro:macro>
-  <xacro:macro name="set_all_wheel_frictions" params="prefix">
-    <xacro:set_wheel_friction link="${prefix}left_wheel_link" friction="200"/>
-    <xacro:set_wheel_friction link="${prefix}right_wheel_link" friction="200"/>
-    <xacro:set_wheel_friction link="${prefix}fl_caster_wheel_link" friction="1"/>
-    <xacro:set_wheel_friction link="${prefix}fr_caster_wheel_link" friction="1"/>
-    <xacro:set_wheel_friction link="${prefix}bl_caster_wheel_link" friction="1"/>
-    <xacro:set_wheel_friction link="${prefix}br_caster_wheel_link" friction="1"/>
-  </xacro:macro>
  <!-- See https://github.com/ros-simulation/gazebo_ros_pkgs/wiki/ROS-2-Migration:-P3D for ros2 information -->
   <xacro:macro name="p3d_base_controller" params="prefix">

File: mir_description/urdf/include/mir_100_v1.urdf.xacro (robot description, xacro)
@@ -6,6 +6,16 @@
   <xacro:include filename="$(find mir_description)/urdf/include/mir_100.transmission.xacro" />
   <xacro:include filename="$(find mir_description)/urdf/include/sick_s300.urdf.xacro" />
+  <xacro:include filename="$(find mir_description)/urdf/include/wheel.urdf.xacro" />
+  <xacro:include filename="$(find mir_description)/urdf/include/caster.urdf.xacro" />
   <xacro:property name="deg_to_rad" value="0.017453293" />
-  <xacro:property name="mir_100_base_mass" value="58.0" />
+  <!-- The inertia for the MiR platform is intentionally chosen to be smaller than
+       the bounding box and also shifted a bit to the back, because most of the mass
+       is in the lower center back (because of the batteries). -->
+  <xacro:property name="mir_base_inertial_x" value="-0.05" />
+  <xacro:property name="mir_base_inertial_y" value="0.0" />
+  <xacro:property name="mir_base_inertial_z" value="0.15" />
+  <xacro:property name="mir_base_inertial_x_length" value="0.50" />
+  <xacro:property name="mir_base_inertial_y_length" value="0.30" />
+  <xacro:property name="mir_base_inertial_z_length" value="0.20" />
   <xacro:property name="mir_100_act_wheel_radius" value="0.0625" />
   <xacro:property name="mir_100_act_wheel_width" value="0.032" />
@@ -23,121 +33,10 @@
   <xacro:property name="mir_100_caster_wheel_base_dy" value="0.203" />
   <xacro:property name="mir_100_caster_wheel_base_dz" value="${mir_100_caster_wheel_radius-mir_100_caster_wheel_dz}" />
+  <!-- MiR 100 complete mass 78.2kg (8.2kg battery) -->
+  <!-- - 2x2kg sick laser = 4kg-->
+  <!-- - 4x caster wheels + rotation link: 4x 1.31 kg -->
+  <!-- - 2x act wheels: 2kg -->
+  <xacro:property name="mir_100_base_mass" value="66.96" />
   <xacro:property name="imu_stdev" value="0.00017" />
-  <xacro:macro name="actuated_wheel" params="prefix  locationprefix locationright">
-    <joint name="${prefix}${locationprefix}_wheel_joint" type="continuous">
-      <origin xyz="0.0 ${-mir_100_act_wheel_dy * locationright} ${mir_100_act_wheel_radius}" rpy="0 0 0" />
-      <parent link="${prefix}base_link" />
-      <child link="${prefix}${locationprefix}_wheel_link" />
-      <axis xyz="0 1 0" />
-      <limit effort="100" velocity="20.0" />
-    </joint>
-    <link name="${prefix}${locationprefix}_wheel_link">
-      <xacro:cylinder_inertial mass="${mir_100_act_wheel_mass}" radius="${mir_100_act_wheel_radius}" length="${mir_100_act_wheel_width}">
-        <origin xyz="0 0 0" rpy="${0.5 * pi} 0 0" />
-      </xacro:cylinder_inertial>
-      <visual>
-        <origin xyz="0 0 0" rpy="0 0 0" />
-        <geometry>
-          <mesh filename="package://mir_description/meshes/visual/wheel.stl" />
-        </geometry>
-        <xacro:insert_block name="material_dark_grey" />
-      </visual>
-      <collision>
-        <origin xyz="0 0 0" rpy="${pi/2} 0 0" />
-        <geometry>
-          <cylinder radius="${mir_100_act_wheel_radius}" length="${mir_100_act_wheel_width}" />
-        </geometry>
-      </collision>
-    </link>
-    <gazebo reference="${prefix}${locationprefix}_wheel_link">
-      <material>Gazebo/DarkGrey</material>
-    </gazebo>
-  </xacro:macro>
-  <xacro:macro name="caster_wheel" params="prefix ns locationprefix locationright wheel_base_dx">
-    <!-- caster hub -->
-    <joint name="${prefix}${locationprefix}_caster_rotation_joint" type="continuous">
-      <origin xyz="${wheel_base_dx} ${-mir_100_caster_wheel_base_dy * locationright} ${mir_100_caster_wheel_base_dz}" rpy="0 0 0" />
-      <parent link="${prefix}base_link" />
-      <child link="${prefix}${locationprefix}_caster_rotation_link" />
-      <axis xyz="0 0 1" />
-      <dynamics damping="0.01" friction="0.0"/>
-    </joint>
-    <gazebo>
-      <plugin name="${locationprefix}_caster_rotation_joint_states" filename="libgazebo_ros_joint_state_publisher.so">
-        <ros>
-          <namespace>${ns}</namespace>
-        </ros>
-        <update_rate>200.0</update_rate>
-        <joint_name>${prefix}${locationprefix}_caster_rotation_joint</joint_name>
-      </plugin>
-    </gazebo>
-    <link name="${prefix}${locationprefix}_caster_rotation_link">
-      <inertial>
-        <!-- <origin xyz="0 0 -0.042500000044" rpy="${0.5 * pi} ${24 * deg_to_rad} ${1.5 * pi}" /> -->
-        <origin xyz="0 0 -0.042500000044" rpy="${24 * deg_to_rad} 0 ${0.5 * pi} " />
-        <mass value="0.3097539019" />
-        <inertia
-          ixx="0.0005844517978"
-          ixy="0"
-          ixz="0"
-          iyy="0.00052872551237"
-          iyz="0"
-          izz="0.00017923555074" />
-      </inertial>
-      <visual>
-        <origin xyz="0 0 0" rpy="0 0 0" />
-        <geometry>
-          <mesh filename="package://mir_description/meshes/visual/caster_wheel_base.stl" />
-        </geometry>
-        <xacro:insert_block name="material_silver" />
-      </visual>
-      <collision>
-        <origin xyz="0 0 0" rpy="0 0 0" />
-        <geometry>
-          <mesh filename="package://mir_description/meshes/collision/caster_wheel_base.stl" />
-        </geometry>
-      </collision>
-    </link>
-    <gazebo reference="${prefix}${locationprefix}_caster_rotation_link">
-      <material>Gazebo/Grey</material>
-    </gazebo>
-    <!-- caster wheel -->
-    <joint name="${prefix}${locationprefix}_caster_wheel_joint" type="continuous">
-      <origin xyz="${mir_100_caster_wheel_dx} ${-mir_100_caster_wheel_dy * locationright} ${mir_100_caster_wheel_dz}" rpy="0 0 0" />
-      <parent link="${prefix}${locationprefix}_caster_rotation_link" />
-      <child link="${prefix}${locationprefix}_caster_wheel_link" />
-      <axis xyz="0 1 0" />
-    </joint>
-    <gazebo>
-      <plugin name="${locationprefix}_caster_wheel_joint_states" filename="libgazebo_ros_joint_state_publisher.so">
-        <ros>
-          <namespace>${ns}</namespace>
-        </ros>
-        <update_rate>200.0</update_rate>
-        <joint_name>${prefix}${locationprefix}_caster_wheel_joint</joint_name>
-      </plugin>
-    </gazebo>
-    <link name="${prefix}${locationprefix}_caster_wheel_link">
-      <xacro:cylinder_inertial mass="${mir_100_caster_wheel_mass}" radius="${mir_100_caster_wheel_radius}" length="${mir_100_caster_wheel_width}">
-        <origin xyz="0 0 0" rpy="${0.5 * pi} 0 0" />
-      </xacro:cylinder_inertial>
-      <visual>
-        <origin xyz="0 0 0" rpy="0 0 0" />
-        <geometry>
-          <mesh filename="package://mir_description/meshes/visual/wheel.stl" />
-        </geometry>
-        <xacro:insert_block name="material_dark_grey" />
-      </visual>
-      <collision>
-        <origin xyz="0 0 0" rpy="${pi/2} 0 0" />
-        <geometry>
-          <cylinder radius="${mir_100_caster_wheel_radius}" length="${mir_100_caster_wheel_width}" />
-        </geometry>
-      </collision>
-    </link>
-    <gazebo reference="${prefix}${locationprefix}_caster_wheel_link">
-      <material>Gazebo/DarkGrey</material>
-    </gazebo>
-  </xacro:macro>
   <xacro:macro name="mir_100" params="prefix ns">
     <link name="${prefix}base_footprint" />
@@ -148,6 +47,6 @@
     </joint>
     <link name="${prefix}base_link">
-      <xacro:box_inertial mass="${mir_100_base_mass}" x="0.9" y="0.58" z="0.3">
-        <origin xyz="${mir_100_act_wheel_dx} 0 0.20" rpy="0 0 0" />
+      <xacro:box_inertial mass="${mir_100_base_mass}" x="${mir_base_inertial_x_length}" y="${mir_base_inertial_y_length}" z="${mir_base_inertial_z_length}">
+        <origin xyz="${mir_base_inertial_x + mir_100_act_wheel_dx} ${mir_base_inertial_y} ${mir_base_inertial_z}" rpy="0 0 0" />
       </xacro:box_inertial>
       <visual>
@@ -234,6 +133,4 @@
     <link name="${prefix}surface"/>
     <xacro:mir_100_wheel_transmissions prefix="${prefix}"/>
-    <!-- set the gazebo friction parameters for the wheels -->
-    <xacro:set_all_wheel_frictions prefix="${prefix}"/>
     <xacro:p3d_base_controller prefix="${prefix}"/>
   </xacro:macro>
