Commit message: fix colors inside gazebo

File: mir_hook_description/urdf/include/cart.urdf.xacro (robot description, xacro)
@@ -1,4 +1,4 @@
 <?xml version="1.0"?>
-<robot xmlns:xacro="http://ros.org/wiki/xacro">
+<robot name="cart" xmlns:xacro="http://ros.org/wiki/xacro">
   <link name="cart_base_link">
   </link>
@@ -9,5 +9,5 @@
       <inertia ixx="0.06608" ixy="0" ixz="0" iyy="0.05242" iyz="1e-05" izz="0.02359"/>
     </inertial>
-    <visual name="visual_back_stabilizer">
+    <visual>
       <xacro:insert_block name="material_silver" />
       <origin xyz="0.00017 0.38637 1.06389" rpy="0 0 0"/>
@@ -15,9 +15,6 @@
         <mesh filename="package://mir_hook_description/meshes/cart/Part__Feature167.stl" scale="1.0 1.0 1.0"/>
       </geometry>
-      <gazebo reference="cart_root">
-        <material>Gazebo/DarkGrey</material>
-      </gazebo>
-    </visual>
-    <visual name="visual_castor_rigid_left_fork">
+    </visual>
+    <visual>
       <xacro:insert_block name="material_silver" />
       <origin xyz="-0.28116 0.33151 -0.06865" rpy="0 0 0"/>
@@ -25,9 +22,6 @@
         <mesh filename="package://mir_hook_description/meshes/cart/Part__Feature082.stl" scale="1.0 1.0 1.0"/>
       </geometry>
-      <gazebo reference="visual_castor_rigid_left_fork">
-        <material>Gazebo/DarkGrey</material>
-      </gazebo>
-    </visual>
-    <visual name="visual_castor_rigid_right_fork">
+    </visual>
+    <visual>
       <xacro:insert_block name="material_silver" />
       <origin xyz="0.28184 0.33151 -0.06865" rpy="0 0 0"/>
@@ -35,9 +29,6 @@
         <mesh filename="package://mir_hook_description/meshes/cart/Part__Feature099.stl" scale="1.0 1.0 1.0"/>
       </geometry>
-      <gazebo reference="visual_castor_rigid_right_fork">
-        <material>Gazebo/DarkGrey</material>
-      </gazebo>
-    </visual>
-    <visual name="visual_castor_swivel_left_top_plate">
+    </visual>
+    <visual>
       <xacro:insert_block name="material_silver" />
       <origin xyz="-0.28133 -0.32949 -0.04313" rpy="0 0 0"/>
@@ -45,9 +36,6 @@
         <mesh filename="package://mir_hook_description/meshes/cart/Part__Feature021.stl" scale="1.0 1.0 1.0"/>
       </geometry>
-      <gazebo reference="visual_castor_swivel_left_top_plate">
-        <material>Gazebo/DarkGrey</material>
-      </gazebo>
-    </visual>
-    <visual name="visual_castor_swivel_right_top_plate">
+    </visual>
+    <visual>
       <xacro:insert_block name="material_silver" />
       <origin xyz="0.28167 -0.32949 -0.04313" rpy="0 0 0"/>
@@ -55,9 +43,6 @@
         <mesh filename="package://mir_hook_description/meshes/cart/Part__Feature116.stl" scale="1.0 1.0 1.0"/>
       </geometry>
-      <gazebo reference="visual_castor_swivel_right_top_plate">
-        <material>Gazebo/DarkGrey</material>
-      </gazebo>
-    </visual>
-    <visual name="visual_container_base">
+    </visual>
+    <visual>
       <xacro:insert_block name="material_silver" />
       <origin xyz="-0.00111 0 0" rpy="0 0 0"/>
@@ -65,9 +50,6 @@
         <mesh filename="package://mir_hook_description/meshes/cart/Part__Feature.stl" scale="1.01559 1.0 1.0"/>
       </geometry>
-      <gazebo reference="visual_container_base">
-        <material>Gazebo/DarkGrey</material>
-      </gazebo>
-    </visual>
-    <visual name="visual_handle_left">
+    </visual>
+    <visual>
       <xacro:insert_block name="material_silver" />
       <origin xyz="-0.31379 -0.43587 0.90411" rpy="0 0 0"/>
@@ -75,9 +57,6 @@
         <mesh filename="package://mir_hook_description/meshes/cart/Part__Feature163.stl" scale="1.0 1.0 1.0"/>
       </geometry>
-      <gazebo reference="visual_handle_left">
-        <material>Gazebo/DarkGrey</material>
-      </gazebo>
-    </visual>
-    <visual name="visual_handle_right">
+    </visual>
+    <visual>
       <xacro:insert_block name="material_silver" />
       <origin xyz="0.31187 -0.43529 0.90415" rpy="0 0 0"/>
@@ -85,9 +64,6 @@
         <mesh filename="package://mir_hook_description/meshes/cart/Part__Feature166.stl" scale="1.0 1.0 1.0"/>
       </geometry>
-      <gazebo reference="visual_handle_right">
-        <material>Gazebo/DarkGrey</material>
-      </gazebo>
-    </visual>
-    <visual name="visual_wire_lattice_left">
+    </visual>
+    <visual>
       <xacro:insert_block name="material_silver" />
       <origin xyz="-0.3407 0.00254 0.70262" rpy="0 0 0"/>
@@ -95,9 +71,6 @@
         <mesh filename="package://mir_hook_description/meshes/cart/Part__Feature162.stl" scale="1.0 1.0 1.0"/>
       </geometry>
-      <gazebo reference="visual_wire_lattice_left">
-        <material>Gazebo/DarkGrey</material>
-      </gazebo>
-    </visual>
-    <visual name="visual_wire_lattice_right">
+    </visual>
+    <visual>
       <xacro:insert_block name="material_silver" />
       <origin xyz="0.34102 0.00291 0.70264" rpy="0 0 0"/>
@@ -105,7 +78,4 @@
         <mesh filename="package://mir_hook_description/meshes/cart/Part__Feature165.stl" scale="1.0 1.0 1.0"/>
       </geometry>
-      <gazebo reference="visual_wire_lattice_right">
-        <material>Gazebo/DarkGrey</material>
-      </gazebo>
     </visual>
   </link>
@@ -116,5 +86,5 @@
       <inertia ixx="3e-05" ixy="0" ixz="0" iyy="2e-05" iyz="0" izz="2e-05"/>
     </inertial>
-    <visual name="visual_castor_rigid_left_wheel">
+    <visual>
       <xacro:insert_block name="material_red" />
       <origin xyz="0 0 0" rpy="0 -1.5708 0"/>
@@ -122,9 +92,6 @@
         <mesh filename="package://mir_hook_description/meshes/cart/Part__Feature066.stl" scale="1.0 1.0 1.0"/>
       </geometry>
-      <gazebo reference="castor_rigid_left_wheel">
-        <material>Gazebo/DarkGrey</material>
-      </gazebo>
-    </visual>
-    <collision name="collision_castor_rigid_left_wheel">
+    </visual>
+    <collision>
       <origin xyz="-5e-05 0 0" rpy="0 0 0"/>
       <geometry>
@@ -139,5 +106,5 @@
       <inertia ixx="3e-05" ixy="0" ixz="0" iyy="2e-05" iyz="0" izz="2e-05"/>
     </inertial>
-    <visual name="visual_castor_rigid_right_wheel">
+    <visual>
       <xacro:insert_block name="material_red" />
       <origin xyz="0 0 0" rpy="0 -1.5708 0"/>
@@ -145,9 +112,6 @@
         <mesh filename="package://mir_hook_description/meshes/cart/Part__Feature083.stl" scale="1.0 1.0 1.0"/>
       </geometry>
-      <gazebo reference="$castor_rigid_right_wheel">
-        <material>Gazebo/DarkGrey</material>
-      </gazebo>
-    </visual>
-    <collision name="collision_castor_rigid_right_wheel">
+    </visual>
+    <collision>
       <origin xyz="-5e-05 0 0" rpy="0 0 0"/>
       <geometry>
@@ -162,5 +126,5 @@
       <inertia ixx="2e-05" ixy="0" ixz="0" iyy="2e-05" iyz="0" izz="2e-05"/>
     </inertial>
-    <visual name="visual_castor_swivel_left_fork">
+    <visual>
       <xacro:insert_block name="material_silver" />
       <origin xyz="-0.00547 -0.01599 -0.02516" rpy="0 0 0"/>
@@ -168,9 +132,6 @@
         <mesh filename="package://mir_hook_description/meshes/cart/Part__Feature022.stl" scale="1.0 1.0 1.0"/>
       </geometry>
-      <gazebo reference="castor_swivel_left_fork">
-        <material>Gazebo/DarkGrey</material>
-      </gazebo>
-    </visual>
-    <collision name="collision_castor_swivel_left_fork">
+    </visual>
+    <collision>
       <origin xyz="0.00029 -0.01005 -0.03671" rpy="0 0 0"/>
       <geometry>
@@ -185,5 +146,5 @@
       <inertia ixx="3e-05" ixy="0" ixz="0" iyy="2e-05" iyz="0" izz="2e-05"/>
     </inertial>
-    <visual name="visual_castor_swivel_left_wheel">
+    <visual>
       <xacro:insert_block name="material_red" />
       <origin xyz="0 0 -5e-05" rpy="0.50265 -1.5708 0"/>
@@ -191,9 +152,6 @@
         <mesh filename="package://mir_hook_description/meshes/cart/Part__Feature006.stl" scale="1.0 1.0 1.0"/>
       </geometry>
-      <gazebo reference="castor_swivel_left_wheel">
-        <material>Gazebo/DarkGrey</material>
-      </gazebo>
-    </visual>
-    <collision name="collision_castor_swivel_left_wheel">
+    </visual>
+    <collision>
       <origin xyz="0 0 0" rpy="0 0 0"/>
       <geometry>
@@ -208,5 +166,5 @@
       <inertia ixx="2e-05" ixy="0" ixz="0" iyy="2e-05" iyz="0" izz="2e-05"/>
     </inertial>
-    <visual name="visual_castor_swivel_right_fork">
+    <visual>
       <xacro:insert_block name="material_silver" />
       <origin xyz="-0.00589 -0.01692 -0.02589" rpy="0 0 0"/>
@@ -214,9 +172,6 @@
         <mesh filename="package://mir_hook_description/meshes/cart/Part__Feature117.stl" scale="1.0 1.0 1.0"/>
       </geometry>
-      <gazebo reference="castor_swivel_right_fork">
-        <material>Gazebo/DarkGrey</material>
-      </gazebo>
-    </visual>
-    <collision name="collision_castor_swivel_right_fork">
+    </visual>
+    <collision>
       <origin xyz="0.00107 -0.00955 -0.03667" rpy="0 0 0"/>
       <geometry>
@@ -231,5 +186,5 @@
       <inertia ixx="3e-05" ixy="0" ixz="0" iyy="2e-05" iyz="0" izz="2e-05"/>
     </inertial>
-    <visual name="visual_castor_swivel_right_wheel">
+    <visual>
       <xacro:insert_block name="material_red" />
       <origin xyz="0 0 5e-05" rpy="0 -1.5708 0"/>
@@ -237,15 +192,34 @@
         <mesh filename="package://mir_hook_description/meshes/cart/Part__Feature083_001.stl" scale="1.0 1.0 1.0"/>
       </geometry>
-      <gazebo reference="castor_swivel_right_wheel">
-        <material>Gazebo/DarkGrey</material>
-      </gazebo>
-    </visual>
-    <collision name="collision_castor_swivel_right_wheel">
-      <origin xyz="0 0 0" rpy="0 0 0"/>
-      <geometry>
-        <sphere radius="0.0495"/>
-      </geometry>
-    </collision>
-  </link>
+    </visual>
+    <collision>
+      <origin xyz="0 0 0" rpy="0 0 0"/>
+      <geometry>
+        <sphere radius="0.0495"/>
+      </geometry>
+    </collision>
+  </link>
+  <gazebo reference="castor_rigid_left_wheel">
+    <material>Gazebo/Red</material>
+  </gazebo>
+  <gazebo reference="castor_rigid_right_wheel">
+    <material>Gazebo/Red</material>
+  </gazebo>
+  <gazebo reference="castor_swivel_left_wheel">
+    <material>Gazebo/Red</material>
+  </gazebo>
+  <gazebo reference="castor_swivel_right_wheel">
+    <material>Gazebo/Red</material>
+  </gazebo>
+  <!-- silver ~ (light) Gazebo/Grey -->
+  <gazebo reference="castor_swivel_right_fork">
+    <material>Gazebo/Grey</material>
+  </gazebo>
+  <gazebo reference="castor_swivel_left_fork">
+    <material>Gazebo/Grey</material>
+  </gazebo>
+  <gazebo reference="cart_root">
+    <material>Gazebo/Grey</material>
+  </gazebo>
   <joint name="castor_rigid_left_wheel_joint" type="continuous">
     <origin xyz="-0.28128 0.33151 -0.11689" rpy="0 1.5708 0"/>

File: mir_hook_description/urdf/include/hook.urdf.xacro (robot description, xacro)
@@ -8,5 +8,5 @@
       <inertia ixx="0.0102801" ixy="0.0005188" ixz="-0.0035496" iyy="0.0089798" iyz="-7.18e-05" izz="0.0049397" />
     </inertial>
-    <visual name="visual_carriage">
+    <visual>
       <origin xyz="-0.0345127 -0.0820147 3.1e-06" rpy="-1.5707964 0 0" />
       <geometry>
@@ -14,9 +14,6 @@
       </geometry>
       <xacro:insert_block name="material_grey" />
-      <gazebo reference="carriage">
-        <material>Gazebo/DarkGrey</material>
-      </gazebo>
-    </visual>
-    <visual name="visual_container_crawler">
+    </visual>
+    <visual>
       <origin xyz="-0.2067981 -0.2896011 3e-06" rpy="-1.5707964 0 0" />
       <geometry>
@@ -24,67 +21,40 @@
       </geometry>
       <xacro:insert_block name="material_grey" />
-      <gazebo reference="carriage">
-        <material>Gazebo/DarkGrey</material>
-      </gazebo>
-    </visual>
-    <visual name="visual_container_lock">
+    </visual>
+    <visual>
       <origin xyz="-0.1818805 -0.180375 -0.000269" rpy="-1.5707964 0 0" />
       <geometry>
         <mesh filename="package://mir_hook_description/meshes/hook/container_lock.stl" scale="1.0 1.0 1.0" />
       </geometry>
-      <gazebo reference="carriage">
-        <xacro:insert_block name="material_grey" />
-        <material>Gazebo/DarkGrey</material>
-      </gazebo>
-    </visual>
-    <visual name="visual_fork_base">
+    </visual>
+    <visual>
       <origin xyz="-0.1448901 -0.2715 3.2e-06" rpy="-1.5707964 0 0" />
       <geometry>
         <mesh filename="package://mir_hook_description/meshes/hook/fork_base.stl" scale="1.0 1.0 1.0" />
       </geometry>
-      <gazebo reference="carriage">
-        <xacro:insert_block name="material_grey" />
-        <material>Gazebo/DarkGrey</material>
-      </gazebo>
-    </visual>
-    <visual name="visual_tilt_actuator_cylinder">
+    </visual>
+    <visual>
       <origin xyz="-0.1676646 -0.1944744 0.0017018" rpy="-1.5707964 0 0" />
       <geometry>
         <mesh filename="package://mir_hook_description/meshes/hook/Part__Feature079.stl" scale="1.0000001 1.0 1.0000001" />
       </geometry>
-      <gazebo reference="carriage">
-        <material>Gazebo/DarkGrey</material>
-        <xacro:insert_block name="material_grey" />
-      </gazebo>
-    </visual>
-    <visual name="visual_tilt_actuator_motor">
+    </visual>
+    <visual>
       <origin xyz="-0.1158853 -0.0953563 0.0017019" rpy="-1.5707964 0 0" />
       <geometry>
         <mesh filename="package://mir_hook_description/meshes/hook/Part__Feature078.stl" scale="1.0000001 1.0 1.0000001" />
       </geometry>
-      <gazebo reference="carriage">
-        <material>Gazebo/DarkGrey</material>
-        <xacro:insert_block name="material_grey" />
-      </gazebo>
-    </visual>
-    <visual name="visual_tilt_arm_lower">
+    </visual>
+    <visual>
       <origin xyz="-0.13785 -0.3212596 3e-06" rpy="-1.5707964 0 0" />
       <geometry>
         <mesh filename="package://mir_hook_description/meshes/hook/tilt_arm_lower.stl" scale="1.0 1.0 1.0" />
       </geometry>
-      <gazebo reference="carriage">
-        <material>Gazebo/DarkGrey</material>
-        <xacro:insert_block name="material_grey" />
-      </gazebo>
-    </visual>
-    <visual name="visual_tilt_arm_upper">
+    </visual>
+    <visual>
       <origin xyz="-0.1404309 -0.2453349 3e-06" rpy="-1.5707964 0 0" />
       <geometry>
         <mesh filename="package://mir_hook_description/meshes/hook/Part__Feature158.stl" scale="1.0 1.0 1.0" />
       </geometry>
-      <gazebo reference="carriage">
-        <material>Gazebo/DarkGrey</material>
-        <xacro:insert_block name="material_grey" />
-      </gazebo>
     </visual>
     <collision name="collision_carriage_1">
@@ -233,5 +203,5 @@
       <inertia ixx="0.0003373" ixy="-0.0006013" ixz="0" iyy="0.0014916" iyz="0" izz="0.0012083" />
     </inertial>
-    <visual name="visual_lift_arm_lower">
+    <visual>
       <origin xyz="-0.2092547 0.1067384 3.3e-05" rpy="-1.5707964 0 0" />
       <geometry>
@@ -239,7 +209,4 @@
       </geometry>
       <xacro:insert_block name="material_grey" />
-      <gazebo reference="lift_arm_lower">
-        <material>Gazebo/DarkGrey</material>
-      </gazebo>
     </visual>
     <collision name="collision_lift_arm_lower">
@@ -252,28 +219,35 @@
   <link name="lift_arm_upper">
     <inertial>
-      <origin xyz="-0.1397772 0.0769129 -9.87e-05" rpy="0 0 0" />
+      <origin xyz="-0.1397772 0.0769129 0.0" rpy="0 0 0" />
       <mass value="2.2" />
       <inertia ixx="0.0009413" ixy="-0.0006054" ixz="0.0005665" iyy="0.0032542" iyz="-1.06e-05" izz="0.0025802" />
     </inertial>
-    <visual name="visual_emergency_stop">
+    <visual>
+      <origin xyz="-0.2092544 0.1027477 0" rpy="-1.5707964 0 0" />
+      <geometry>
+        <mesh filename="package://mir_hook_description/meshes/hook/lift_arm_upper.stl" scale="1.0 1.0 1.0" />
+      </geometry>
+      <xacro:insert_block name="material_grey" />
+    </visual>
+    <collision name="collision_lift_arm_upper">
+      <origin xyz="-0.2092544 0.1062098 0" rpy="-1.5707964 0 -0.4712389" />
+      <geometry>
+        <box size="0.4483504 0.0915001 0.0251618" />
+      </geometry>
+    </collision>
+  </link>
+  <link name="emergency_stop_arm">
+    <inertial>
+      <origin xyz="-0.1397772 0.0769129 0.0" rpy="0 0 0" />
+      <mass value="0.05" />
+      <inertia ixx="0.0009413" ixy="-0.0006054" ixz="0.0005665" iyy="0.0032542" iyz="-1.06e-05" izz="0.0025802" />
+    </inertial>
+    <visual>
       <xacro:insert_block name="material_red" />
-      <origin xyz="-0.0732943 0.0745365 -5.57e-05" rpy="-1.5707964 0 0" />
+      <!-- origin xyz="-0.0732943 0.0745365 0.0" rpy="-1.5707964 0 0" /-->
+      <origin xyz="-0.0732943 0.2145365 0.0" rpy="-1.5707964 0 0" />
       <geometry>
         <mesh filename="package://mir_hook_description/meshes/hook/emergency_stop.stl" scale="1.0 1.0 1.0" />
       </geometry>
-      <gazebo reference="lift_arm_upper">
-        <xacro:insert_block name="material_grey" />
-        <material>Gazebo/DarkGrey</material>
-      </gazebo>
-    </visual>
-    <visual name="visual_lift_arm_upper">
-      <origin xyz="-0.2092544 0.1027477 0" rpy="-1.5707964 0 0" />
-      <geometry>
-        <mesh filename="package://mir_hook_description/meshes/hook/lift_arm_upper.stl" scale="1.0 1.0 1.0" />
-      </geometry>
-      <xacro:insert_block name="material_grey" />
-      <gazebo reference="lift_arm_upper">
-        <material>Gazebo/DarkGrey</material>
-      </gazebo>
     </visual>
     <collision name="collision_emergency_stop">
@@ -281,10 +255,4 @@
       <geometry>
         <cylinder radius="0.0200511" length="0.0454842" />
-      </geometry>
-    </collision>
-    <collision name="collision_lift_arm_upper">
-      <origin xyz="-0.2092544 0.1062098 0" rpy="-1.5707964 0 -0.4712389" />
-      <geometry>
-        <box size="0.4483504 0.0915001 0.0251618" />
       </geometry>
     </collision>
@@ -296,5 +264,5 @@
       <inertia ixx="0.0001287" ixy="-3.9e-06" ixz="3.2e-05" iyy="0.0001894" iyz="4.65e-05" izz="8.17e-05" />
     </inertial>
-    <visual name="visual_lift_actuator_cylinder">
+    <visual>
       <origin xyz="-0.1810796 0.1424212 8.3e-06" rpy="-1.5707964 0 0" />
       <geometry>
@@ -302,9 +270,6 @@
       </geometry>
       <xacro:insert_block name="material_grey" />
-      <gazebo reference="lift_motor_joint">
-        <material>Gazebo/DarkGrey</material>
-      </gazebo>
-    </visual>
-    <visual name="visual_lift_actuator_motor">
+    </visual>
+    <visual>
       <origin xyz="-0.0706371 0.0612726 3.1e-06" rpy="-1.5707964 0 0" />
       <geometry>
@@ -312,7 +277,4 @@
       </geometry>
       <xacro:insert_block name="material_grey" />
-      <gazebo reference="lift_motor_joint">
-        <material>Gazebo/DarkGrey</material>
-      </gazebo>
     </visual>
     <collision name="collision_lift_actuator_cylinder">
@@ -335,12 +297,9 @@
       <inertia ixx="0.0013133" ixy="0.000168" ixz="5e-07" iyy="0.0014023" iyz="-1.4e-06" izz="0.000605" />
     </inertial>
-    <visual name="visual_pan_motor">
+    <visual>
       <origin xyz="-0.0200243 -0.0003519 -0.0032138" rpy="0 0 0" />
       <geometry>
         <mesh filename="package://mir_hook_description/meshes/hook/pan_motor.stl" scale="1.0 1.0 1.0" />
       </geometry>
-      <gazebo reference="pan_motor">
-        <material>Gazebo/DarkGrey</material>
-      </gazebo>
       <xacro:insert_block name="material_grey" />
     </visual>
@@ -358,5 +317,5 @@
       <inertia ixx="0.0132281" ixy="-0.0003299" ixz="2.77e-05" iyy="0.0183048" iyz="-9.9e-06" izz="0.0244622" />
     </inertial>
-    <visual name="visual_frame">
+    <visual>
       <xacro:insert_block name="material_white" />
       <origin xyz="-0.0690002 -2.2e-06 0.1547746" rpy="0 0 0" />
@@ -364,7 +323,4 @@
         <mesh filename="package://mir_hook_description/meshes/hook/frame.stl" scale="1.0 1.0 1.0" />
       </geometry>
-      <gazebo reference="hook_root">
-        <material>Gazebo/DarkGrey</material>
-      </gazebo>
     </visual>
     <collision name="collision_frame_1">
@@ -417,4 +373,25 @@
     </collision>
   </link>
+  <gazebo reference="hook_root">
+    <material>Gazebo/White</material>
+  </gazebo>
+  <gazebo reference="carriage">
+    <material>Gazebo/DarkGrey</material>
+  </gazebo>
+  <gazebo reference="lift_arm_lower">
+    <material>Gazebo/DarkGrey</material>
+  </gazebo>
+  <gazebo reference="lift_arm_upper">
+    <material>Gazebo/DarkGrey</material>
+  </gazebo>
+  <gazebo reference="lift_motor_joint">
+    <material>Gazebo/DarkGrey</material>
+  </gazebo>
+  <gazebo reference="pan_motor">
+    <material>Gazebo/DarkGrey</material>
+  </gazebo>
+  <gazebo reference="emergency_stop_arm">
+    <material>Gazebo/Red</material>
+  </gazebo>
   <joint name="hook_root" type="fixed">
     <origin xyz="0.110500 -0.00587 0.347745" rpy="0 0 0" />
@@ -435,4 +412,11 @@
     <parent link="pan_motor" />
     <child link="lift_arm_lower" />
+    <axis xyz="0 0 1.0" />
+    <limit lower="0" upper="0.5235988" effort="100.0" velocity="6.0" />
+  </joint>
+  <joint name="emergency_stop_arm" type="fixed">
+    <origin xyz="-0.077511 3.3e-05 -0.0564022" rpy="1.5707964 0 0" />
+    <parent link="pan_motor" />
+    <child link="emergency_stop_arm" />
     <axis xyz="0 0 1.0" />
     <limit lower="0" upper="0.5235988" effort="100.0" velocity="6.0" />

File: mir_hook_description/urdf/include/mir_hook_common.urdf.xacro (robot description, xacro)
@@ -9,9 +9,3 @@
     </material>
   </xacro:property>
-  <xacro:property name="material_black">
-    <material name="black">
-      <!-- use a "lighter" black so you can see the outline of the object -->
-      <color rgba="${20/255} ${20/255} ${20/255} 1"/>
-    </material>
-  </xacro:property>
 </robot>
