Commit message: lower hook to match position of cart

File: mir_hook_description/urdf/include/cart.urdf.xacro (robot description, xacro)
@@ -277,5 +277,5 @@
   </joint>
   <joint name="cart_base_link_to_root" type="fixed">
-    <origin xyz="-0.33151 0.0 0.11689" rpy="0.0 0.0 -1.5707"/>
+    <origin xyz="-0.33151 0.0 0.33" rpy="0.0 0.0 -1.5707"/>
     <parent link="cart_base_link"/>
     <child link="cart_root"/>

File: mir_hook_description/urdf/include/hook.urdf.xacro (robot description, xacro)
@@ -1,5 +1,4 @@
 <?xml version="1.0"?>
 <robot xmlns:xacro="http://ros.org/wiki/xacro">
-  <!-- hook -->
   <link name="carriage">
     <inertial>
@@ -85,5 +84,5 @@
       <origin xyz="-0.2129726 -0.3028729 0.132826" rpy="-1e-07 0 0.8045967" />
       <geometry>
-        <cylinder radius="0.05733" length="0.00544" />
+        <box size="0.11466 0.06084 0.00544" />
       </geometry>
     </collision>
@@ -91,4 +90,5 @@
       <origin xyz="-0.212973 -0.3028729 -0.132826" rpy="-1e-07 0 0.8045968" />
       <geometry>
+        <!--box size="0.11466 0.06084 0.00544" /-->
         <cylinder radius="0.05733" length="0.00544" />
       </geometry>
@@ -260,10 +260,10 @@
   <link name="lift_motor_joint">
     <inertial>
-      <origin xyz="-0.0288321 0.0338943 0.011049" rpy="0 0 0" />
+      <origin xyz="-0.0294563 0.0338943 -0.0067328" rpy="0 0 0" />
       <mass value="0.55" />
-      <inertia ixx="0.0001287" ixy="-3.9e-06" ixz="3.2e-05" iyy="0.0001894" iyz="4.65e-05" izz="8.17e-05" />
-    </inertial>
-    <visual>
-      <origin xyz="-0.1810796 0.1424212 8.3e-06" rpy="-1.5707964 0 0" />
+      <inertia ixx="2.07e-05" ixy="1.02e-05" ixz="2.37e-05" iyy="9.31e-05" iyz="4.58e-05" izz="7.67e-05" />
+    </inertial>
+    <visual>
+      <origin xyz="-0.1339298 0.1073225 8.3e-06" rpy="-1.5707964 0 0" />
       <geometry>
         <mesh filename="package://mir_hook_description/meshes/hook/Part__Feature063.stl" scale="1.0 1.0 1.0" />
@@ -279,5 +279,5 @@
     </visual>
     <collision name="collision_lift_actuator_cylinder">
-      <origin xyz="-0.1900736 0.1490457 3.1e-06" rpy="-1.5707963 0 -2.2375119" />
+      <origin xyz="-0.1429238 0.1139471 3.1e-06" rpy="-1.5707964 0 -2.2375121" />
       <geometry>
         <cylinder radius="0.0096713" length="0.1076295" />
@@ -402,5 +402,5 @@
   </joint>
   <joint name="carriage" type="fixed">
-    <origin xyz="-0.418597 0.213663 3e-05" rpy="0 0 0" />
+    <origin xyz="-0.418597 0.213663 3e-05" rpy="0 0 -0.4712389" />
     <parent link="lift_arm_lower" />
     <child link="carriage" />
@@ -409,5 +409,5 @@
   </joint>
   <joint name="lift_arm_lower" type="fixed">
-    <origin xyz="-0.077511 3.3e-05 -0.0564022" rpy="1.5707964 0 0" />
+    <origin xyz="-0.077511 3.3e-05 -0.0564022" rpy="1.5707964 -0.4712389 0" />
     <parent link="pan_motor" />
     <child link="lift_arm_lower" />
@@ -416,5 +416,5 @@
   </joint>
   <joint name="emergency_stop_arm" type="fixed">
-    <origin xyz="-0.077511 3.3e-05 -0.0564022" rpy="1.5707964 0 0" />
+    <origin xyz="-0.077511 3.3e-05 -0.0564022" rpy="1.5707964 -0.4712389 0" />
     <parent link="pan_motor" />
     <child link="emergency_stop_arm" />
@@ -423,5 +423,5 @@
   </joint>
   <joint name="lift_arm_upper" type="fixed">
-    <origin xyz="-0.0775113 0 0.0832461" rpy="1.5707964 0 0" />
+    <origin xyz="-0.0775113 0 0.0832461" rpy="1.5707964 -0.4712389 0" />
     <parent link="pan_motor" />
     <child link="lift_arm_upper" />
@@ -430,5 +430,5 @@
   </joint>
   <joint name="lift_motor_joint" type="fixed">
-    <origin xyz="-0.1756014 0.1282467 3e-05" rpy="0 0 0" />
+    <origin xyz="-0.1756014 0.1282466 3e-05" rpy="0 0 -0.111304" />
     <parent link="lift_arm_lower" />
     <child link="lift_motor_joint" />
