Commit message: Move emergency button collision position + inertial
inertial was computed using cylinder_inertial in
mir_description/common_properties.urdf.xacro

File: mir_hook_description/urdf/include/hook.urdf.xacro (robot description, xacro)
@@ -239,7 +239,7 @@
   <link name="emergency_stop_arm">
     <inertial>
-      <origin xyz="-0.1397772 0.0769129 0.0" rpy="0 0 0" />
+      <origin xyz="-0.0732943 0.2145365 0.0" rpy="-1.5707964 0 -0.4712389" />
       <mass value="0.05" />
-      <inertia ixx="0.0009413" ixy="-0.0006054" ixz="0.0005665" iyy="0.0032542" iyz="-1.06e-05" izz="0.0025802" />
+      <inertia ixx="1.3645629055371196e-05" ixy="0.0" ixz="0.0" iyy="1.3645629055371196e-05" iyz="0.0" izz="1.0051165280249999e-05" />
     </inertial>
     <visual>
@@ -252,5 +252,5 @@
     </visual>
     <collision name="collision_emergency_stop">
-      <origin xyz="-0.0769995 0.0721075 -0.0002136" rpy="-1.5707964 0 -0.4712389" />
+      <origin xyz="-0.0732943 0.2145365 0.0" rpy="-1.5707964 0 -0.4712389" />
       <geometry>
         <cylinder radius="0.0200511" length="0.0454842" />

Commit message: Fix hook joint limits

File: mir_hook_description/urdf/include/hook.urdf.xacro (robot description, xacro)
@@ -439,5 +439,5 @@
   <joint name="pan_motor_joint" type="revolute">
     <axis xyz="0 0 1.0" />
-    <limit lower="-1.0" upper="1.0" effort="100.0" velocity="0" />
+    <limit lower="${-pi/2}" upper="${pi/2}" effort="100.0" velocity="0" />
     <origin xyz="-0.067 -3e-06 0.1383631" rpy="0 0 0" />
     <parent link="hook_root" />
